File: z9-pdm/power.kicad_sch (KiCad schematic)
At the start: 28 parts, among them U1 B0505XT-1WR3, U22 TLV76733DRVx, U6 LMR14206

Commit message: cleanup - change fus as test to shorten vale
Parts:
- F3: value Fuse_16V_500mA_100A_1A_150mΩ_0805_PTC_Resettable_Fuses_ROHS -> Fuse_16V_500mA_100A_1A_150mΩ_0805_PTC
Other:
- note added: "Need power flags after fuses/connectors etc for DRC"
Changed lines of the file:
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@@
+		)
+	)
+	(text "Need power flags after fuses/connectors etc for DRC"
+		(exclude_from_sim no)
+		(at 69.85 22.098 0)
+		(effects
+			(font
+				(size 1.27 1.27)
+			)
 		)
 	)
@@
 	)
 	(symbol
+		(lib_name "Fuse_16V_500mA_100A_1A_150mΩ_0805_PTC_Resettable_Fuses_ROHS_1")
 		(lib_id "dnt_global:Fuse_16V_500mA_100A_1A_150mΩ_0805_PTC_Resettable_Fuses_ROHS")
 		(at 90.17 139.7 90)
@@
 		(on_board yes)
 		(dnp no)
-		(fields_autoplaced yes)
 		(property "Reference" "F3"
 			(at 90.17 133.35 90)
@@
 			)
 		)
-		(property "Value" "Fuse_16V_500mA_100A_1A_150mΩ_0805_PTC_Resettable_Fuses_ROHS"
-			(at 90.17 135.89 90)
-			(effects
-				(font
+		(property "Value" "Fuse_16V_500mA_100A_1A_150mΩ_0805_PTC"
+			(at 89.408 128.016 90)
+			(effects
+				(font
