File: z9-pdm/can.kicad_sch (KiCad schematic)
At the start: 6 parts, among them U2 ISO1042-Q1

Commit message: x
Parts:
- JP2: footprint (none) -> Jumper:SolderJumper-2_P1.3mm_Bridged2Bar_Pad1.0x1.5mm
Changed lines of the file:
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@@
 			)
 		)
-		(property "Footprint" ""
+		(property "Footprint" "Jumper:SolderJumper-2_P1.3mm_Bridged2Bar_Pad1.0x1.5mm"
 			(at 144.78 82.55 0)
 			(effects

Commit message: x
Parts:
- JP2: footprint Jumper:SolderJumper-2_P1.3mm_Bridged2Bar_Pad1.0x1.5mm -> (none)
Changed lines of the file:
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@@
 			)
 		)
-		(property "Footprint" "Jumper:SolderJumper-2_P1.3mm_Bridged2Bar_Pad1.0x1.5mm"
+		(property "Footprint" ""
 			(at 144.78 82.55 0)
 			(effects
