File: z9-pdm/can.kicad_sch (KiCad schematic)
At the start: 6 parts, among them U2 ISO1042-Q1

Commit message: pdm sch drc clean
Parts:
- removed C22, C25: 100nF, PCM_JLCPCB:C_0603, symbol PCM_JLCPCB-Capacitors:0603,100nF
- removed C24: 10uF, PCM_JLCPCB:C_0603, symbol PCM_JLCPCB-Capacitors:0603,10uF,(2)
- removed JP2: SolderJumper_2_Bridged, symbol Jumper:SolderJumper_2_Bridged
- removed R1: 120R, Resistor_SMD:R_0805_2012Metric, symbol dnt_global:Resisitor_120R_0805
- removed U2: ISO1042-Q1, Package_SO:SOIC-8_7.5x5.85mm_P1.27mm, symbol dnt_global:ISO1042-Q1
Other:
- note removed: "Near VCC1"
- note removed: "Near VCC2"
