File: z9-pdm/stm32.kicad_sch (KiCad schematic)
At the start: 56 parts, among them J4 Conn_ST_STDC14, J5 DF40HC3.0-100DS-0.4V51, J7 Conn_TagConnect_2070, SW1 Tactile Button, 160gf, SW2 Tactile Button, 160gf, U3 STM32F427V_G-I_Tx, X1 8MHz 20pF

Commit message: pdm sch drc clean
Parts:
- RN1, RN2: Part # CAT16-1001F4LF -> (none)
