File: z9-pdm/vn9e30.kicad_sch (KiCad schematic)
At the start: 3 parts, among them U5 VN9E30F

Commit message: x
Parts:
- U5: footprint dnt:QFN6x6_VN9D30_STM-cleanimport -> dnt:QFN6x6_VN9D30_STM; symbol dnt_global:VN9E30F -> dnt_global:VN9D30Q100F
Connections:
- net OUTPUT0: now also U5.3 (OUTPUT0)
- net OUTPUT1: now also U5.31 (OUTPUT1)
- net OUTPUT2: now also U5.29 (OUTPUT2)
- net OUTPUT3: now also U5.27 (OUTPUT3)
- net OUTPUT4: now also U5.25 (OUTPUT4)
- net OUTPUT5: now also U5.21 (OUTPUT5)
Other:
- moved on the sheet: R23, R24

Commit message: x
Changed lines of the file:
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@@
 		(pin "8"
-		)
-		(pin "35"
 		)
 		(pin "2"
@@
 		(pin "7"
 		)
-		(pin "37"
-		)
-		(pin "34"
-		)
 		(pin "21"
 		)
 		(pin "23"
 		)
-		(pin "36"
-		)
 		(pin "27"
