File: z9-pdm/_autosave-power.kicad_sch (KiCad schematic)
At the start: 28 parts, among them U1 B0505XT-1WR3, U22 TLV76733DRVx, U6 LMR14206

Commit message: pdm sch drc clean
Parts:
- D13: value Diode - Schotty V1P6-M3/H 60V 1A -> Schotty V1P6-M3/H 60V 1A
Other:
- moved on the sheet: F2
Changed lines of the file:
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@@
 	(wire
 		(pts
-			(xy 204.47 34.29) (xy 207.01 34.29)
+			(xy 204.47 34.29) (xy 219.71 34.29)
 		)
 		(stroke
@@
 	(wire
 		(pts
-			(xy 214.63 34.29) (xy 246.38 34.29)
+			(xy 227.33 34.29) (xy 246.38 34.29)
 		)
 		(stroke
@@
 			)
 		)
-		(property "Value" "Diode - Schotty V1P6-M3/H 60V 1A"
-			(at 182.626 54.102 90)
+		(property "Value" "Schotty V1P6-M3/H 60V 1A"
+			(at 178.054 76.708 90)
 			(effects
 				(font
@@
 	(symbol
 		(lib_id "dnt_global:Fuse_16V_500mA_100A_1A_150mΩ_0805_PTC_Resettable_Fuses_ROHS")
-		(at 210.82 34.29 90)
+		(at 223.52 34.29 90)
 		(unit 1)
 		(exclude_from_sim no)
@@
 		(fields_autoplaced yes)
 		(property "Reference" "F2"
-			(at 210.82 27.94 90)
+			(at 223.52 27.94 90)
 			(effects
 				(font
@@
 		)
 		(property "Value" "Fuse_16V_500mA_100A_1A_150mΩ_0805_PTC_Resettable_Fuses_ROHS"
-			(at 210.82 30.48 90)
-			(effects
-				(font
-					(size 1.27 1.27)
-				)
+			(at 223.52 30.48 90)
+			(effects
+				(font
+					(size 1.27 1.27)
+				)
+				(hide yes)
 			)
 		)
 		(property "Footprint" "Fuse:Fuse_0805_2012Metric"
-			(at 210.82 36.068 90)
+			(at 223.52 36.068 90)
 			(effects
 				(font
@@
 		)
 		(property "Datasheet" "~"
-			(at 210.82 34.29 0)
+			(at 223.52 34.29 0)
 			(effects
 				(font
@@
 		)
 		(property "Description" "Fuse"
-			(at 210.82 34.29 0)
+			(at 223.52 34.29 0)
 			(effects
 				(font
@@
 		)
 		(property "LCSC" "C2833485"
-			(at 210.82 34.29 0)
+			(at 223.52 34.29 0)
 			(effects
 				(font
@@
 		)
 		(property "Order" ""
-			(at 210.82 34.29 90)
+			(at 223.52 34.29 90)
 			(effects
 				(font
@@
 		)
 		(property "PN" ""
-			(at 210.82 34.29 90)
+			(at 223.52 34.29 90)
 			(effects
 				(font
@@
 		)
 		(property "Part Number" ""
-			(at 210.82 34.29 90)
+			(at 223.52 34.29 90)
 			(effects
 				(font
@@
 		)
 		(property "Part#" ""
-			(at 210.82 34.29 90)
+			(at 223.52 34.29 90)
 			(effects
 				(font
@@
 		)
 		(property "Vendor" ""
-			(at 210.82 34.29 90)
+			(at 223.52 34.29 90)
 			(effects
 				(font
@@
 		)
 		(property "Voltage" ""
-			(at 210.82 34.29 90)
-			(effects
-				(font
+			(at 223.52 34.29 90)
+			(effects
+				(font
