File: z9-shared/z9-shared.kicad_sch (KiCad schematic)
At the start: 0 parts

Commit message: pdm sch drc clean
Connections:
- no-connect marks 0 -> 10
Other:
- added sheet shared_isolated_can (shared_isolated_can.kicad_sch)
Changed lines of the file:
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@@
 	(generator_version "9.0")
 	(paper "A4")
+	(no_connect
+		(at 83.82 114.3)
+	)
+	(no_connect
+		(at 36.83 78.74)
+	)
+	(no_connect
+		(at 36.83 111.76)
+	)
+	(no_connect
+		(at 36.83 40.64)
+	)
+	(no_connect
+		(at 36.83 43.18)
+	)
+	(no_connect
+		(at 83.82 116.84)
+	)
+	(no_connect
+		(at 36.83 114.3)
+	)
+	(no_connect
+		(at 36.83 116.84)
+	)
+	(no_connect
+		(at 36.83 109.22)
+	)
+	(no_connect
+		(at 36.83 38.1)
+	)
 	(sheet
 		(at 36.83 71.12)
@@
 				)
 			)
+		)
+	)
+	(sheet
+		(at 36.83 106.68)
+		(size 46.99 24.13)
+		(exclude_from_sim no)
+		(in_bom yes)
+		(on_board yes)
+		(dnp no)
+		(fields_autoplaced yes)
+		(stroke
+			(width 0.1524)
+			(type solid)
+		)
+		(fill
+			(color 0 0 0 0.0000)
+		)
+		(property "Sheetname" "shared_isolated_can"
+			(at 36.83 105.9684 0)
+			(show_name yes)
+			(effects
+				(font
+					(size 1.27 1.27)
+				)
+				(justify left bottom)
+			)
+		)
+		(property "Sheetfile" "shared_isolated_can.kicad_sch"
+			(at 36.83 131.3946 0)
+			(show_name yes)
+			(effects
+				(font
+					(size 1.27 1.27)
+				)
+				(justify left top)
+			)
+		)
+		(pin "+5V_ISO" input
+			(at 36.83 111.76 180)
+			(effects
+				(font
+					(size 1.27 1.27)
+				)
+				(justify left)
+			)
+		)
+		(pin "CAN_H" bidirectional
+			(at 36.83 114.3 180)
+			(effects
+				(font
+					(size 1.27 1.27)
+				)
+				(justify left)
+			)
+		)
+		(pin "CAN_L" bidirectional
+			(at 36.83 116.84 180)
+			(effects
+				(font
+					(size 1.27 1.27)
+				)
+				(justify left)
+			)
+		)
+		(pin "CAN_RX" output
+			(at 83.82 114.3 0)
+			(effects
+				(font
+					(size 1.27 1.27)
+				)
+				(justify right)
+			)
+		)
+		(pin "CAN_TX" input
+			(at 83.82 116.84 0)
+			(effects
+				(font
+					(size 1.27 1.27)
+				)
+				(justify right)
+			)
+		)
+		(pin "GND_ISO" input
+			(at 36.83 109.22 180)
+			(effects
+				(font
+					(size 1.27 1.27)
+				)
+				(justify left)
+			)
+		)
+		(instances
+			(project "z9-shared"
+				(path "/09e08bdc-786f-4949-8afc-e02ddbe0502e"
+					(page "4")
+				)
+			)
