File: z9-shared/shared_isolated_can.kicad_sch (KiCad schematic)
At the start: 6 parts, among them U951 ISO1042-Q1

Commit message: annotation issues on shared schematics
Parts:
- renumbered C953 to C?, C951 to C?, C952 to C?, JP951 to JP?, R951 to R?, U951 to U?
Changed lines of the file:
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@@
 		(dnp no)
 		(fields_autoplaced yes)
-		(property "Reference" "#PWR0952"
+		(property "Reference" "#PWR?"
 			(at 128.27 142.24 0)
 			(effects
@@
 				)
 			)
-			(project "z9-shared"
+			(project "z9-pdm"
 				(path "/8d063f79-9282-4820-bcf4-1ff3c006cf08/2345b862-d871-4771-9bee-01079d71c128"
-					(reference "#PWR0952")
+					(reference "#PWR?")
 					(unit 1)
 				)
@@
 		(on_board yes)
 		(dnp no)
-		(property "Reference" "C953"
+		(property "Reference" "C?"
 			(at 185.42 97.79 90)
 			(effects
@@
 				)
 			)
-			(project "z9-shared"
+			(project "z9-pdm"
 				(path "/8d063f79-9282-4820-bcf4-1ff3c006cf08/2345b862-d871-4771-9bee-01079d71c128"
-					(reference "C953")
+					(reference "C?")
 					(unit 1)
 				)
@@
 		(on_board yes)
 		(dnp no)
-		(property "Reference" "R951"
+		(property "Reference" "R?"
 			(at 190.5 73.66 90)
 			(effects
@@
 				)
 			)
-			(project "z9-shared"
+			(project "z9-pdm"
 				(path "/8d063f79-9282-4820-bcf4-1ff3c006cf08/2345b862-d871-4771-9bee-01079d71c128"
-					(reference "R951")
+					(reference "R?")
 					(unit 1)
 				)
@@
 		(on_board yes)
 		(dnp no)
-		(property "Reference" "C951"
+		(property "Reference" "C?"
 			(at 129.54 80.01 90)
 			(effects
@@
 				)
 			)
-			(project "z9-shared"
+			(project "z9-pdm"
 				(path "/8d063f79-9282-4820-bcf4-1ff3c006cf08/2345b862-d871-4771-9bee-01079d71c128"
-					(reference "C951")
+					(reference "C?")
 					(unit 1)
 				)
@@
 		(on_board yes)
 		(dnp no)
-		(property "Reference" "C952"
+		(property "Reference" "C?"
 			(at 169.291 96.6216 0)
 			(effects
@@
 				)
 			)
-			(project "z9-shared"
+			(project "z9-pdm"
 				(path "/8d063f79-9282-4820-bcf4-1ff3c006cf08/2345b862-d871-4771-9bee-01079d71c128"
-					(reference "C952")
+					(reference "C?")
 					(unit 1)
 				)
@@
 		(dnp no)
 		(fields_autoplaced yes)
-		(property "Reference" "#PWR0951"
+		(property "Reference" "#PWR?"
 			(at 78.74 77.47 0)
 			(effects
@@
 				)
 			)
-			(project "z9-shared"
+			(project "z9-pdm"
 				(path "/8d063f79-9282-4820-bcf4-1ff3c006cf08/2345b862-d871-4771-9bee-01079d71c128"
-					(reference "#PWR0951")
+					(reference "#PWR?")
 					(unit 1)
 				)
@@
 		(dnp yes)
 		(fields_autoplaced yes)
-		(property "Reference" "JP951"
+		(property "Reference" "JP?"
 			(at 195.58 64.7699 90)
 			(effects
@@
 				)
 			)
-			(project "z9-shared"
+			(project "z9-pdm"
 				(path "/8d063f79-9282-4820-bcf4-1ff3c006cf08/2345b862-d871-4771-9bee-01079d71c128"
-					(reference "JP951")
+					(reference "JP?")
 					(unit 1)
 				)
@@
 		(dnp no)
 		(fields_autoplaced yes)
-		(property "Reference" "U951"
+		(property "Reference" "U?"
 			(at 146.05 82.55 0)
 			(effects
@@
 				)
 			)
-			(project "z9-shared"
+			(project "z9-pdm"
 				(path "/8d063f79-9282-4820-bcf4-1ff3c006cf08/2345b862-d871-4771-9bee-01079d71c128"
-					(reference "U951")
-					(unit 1)
-				)
+					(reference "U?")
+					(unit 1)
+				)

Commit message: reset shared chematics to correct series
Parts:
- gave numbers to parts that had none: 6
Other:
- note added: "950 series"
- note removed: "use 950 series"
Changed lines of the file:
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@@
 		)
 	)
-	(text "use 950 series "
+	(text "950 series "
 		(exclude_from_sim no)
-		(at 134.112 157.48 0)
+		(at 274.574 162.56 0)
 		(effects
 			(font
@@
 		(dnp no)
 		(fields_autoplaced yes)
-		(property "Reference" "#PWR?"
+		(property "Reference" "#PWR0952"
 			(at 128.27 142.24 0)
 			(effects
@@
 			(project "z9-shared"
 				(path "/09e08bdc-786f-4949-8afc-e02ddbe0502e/a613cbdc-c893-46e2-859f-3c7622690192"
-					(reference "#PWR?")
+					(reference "#PWR0952")
 					(unit 1)
 				)
@@
 		(on_board yes)
 		(dnp no)
-		(property "Reference" "C?"
+		(property "Reference" "C953"
 			(at 185.42 97.79 90)
 			(effects
@@
 			(project "z9-shared"
 				(path "/09e08bdc-786f-4949-8afc-e02ddbe0502e/a613cbdc-c893-46e2-859f-3c7622690192"
-					(reference "C?")
+					(reference "C953")
 					(unit 1)
 				)
@@
 		(on_board yes)
 		(dnp no)
-		(property "Reference" "R?"
+		(property "Reference" "R951"
 			(at 190.5 73.66 90)
 			(effects
@@
 			(project "z9-shared"
 				(path "/09e08bdc-786f-4949-8afc-e02ddbe0502e/a613cbdc-c893-46e2-859f-3c7622690192"
-					(reference "R?")
+					(reference "R951")
 					(unit 1)
 				)
@@
 		(on_board yes)
 		(dnp no)
-		(property "Reference" "C?"
+		(property "Reference" "C951"
 			(at 129.54 80.01 90)
 			(effects
@@
 			(project "z9-shared"
 				(path "/09e08bdc-786f-4949-8afc-e02ddbe0502e/a613cbdc-c893-46e2-859f-3c7622690192"
-					(reference "C?")
+					(reference "C951")
 					(unit 1)
 				)
@@
 		(on_board yes)
 		(dnp no)
-		(property "Reference" "C?"
+		(property "Reference" "C952"
 			(at 169.291 96.6216 0)
 			(effects
@@
 			(project "z9-shared"
 				(path "/09e08bdc-786f-4949-8afc-e02ddbe0502e/a613cbdc-c893-46e2-859f-3c7622690192"
-					(reference "C?")
+					(reference "C952")
 					(unit 1)
 				)
@@
 		(dnp no)
 		(fields_autoplaced yes)
-		(property "Reference" "#PWR?"
+		(property "Reference" "#PWR0951"
 			(at 78.74 77.47 0)
 			(effects
@@
 			(project "z9-shared"
 				(path "/09e08bdc-786f-4949-8afc-e02ddbe0502e/a613cbdc-c893-46e2-859f-3c7622690192"
-					(reference "#PWR?")
+					(reference "#PWR0951")
 					(unit 1)
 				)
@@
 		(dnp yes)
 		(fields_autoplaced yes)
-		(property "Reference" "JP?"
+		(property "Reference" "JP951"
 			(at 195.58 64.7699 90)
 			(effects
@@
 			(project "z9-shared"
 				(path "/09e08bdc-786f-4949-8afc-e02ddbe0502e/a613cbdc-c893-46e2-859f-3c7622690192"
-					(reference "JP?")
+					(reference "JP951")
 					(unit 1)
 				)
@@
 		(dnp no)
 		(fields_autoplaced yes)
-		(property "Reference" "U?"
+		(property "Reference" "U951"
 			(at 146.05 82.55 0)
 			(effects
@@
 			(project "z9-shared"
 				(path "/09e08bdc-786f-4949-8afc-e02ddbe0502e/a613cbdc-c893-46e2-859f-3c7622690192"
-					(reference "U?")
+					(reference "U951")
 					(unit 1)
 				)
