File: z9-shared/shared_usbc.kicad_sch (KiCad schematic)
At the start: 10 parts, among them J801 USB_C_Receptacle_USB2.0_16P

Commit message: x
Other:
- note added: "800 series"
Changed lines of the file:
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@@
 		(title "l8")
+	)
+	(text "800 series"
+		(exclude_from_sim no)
+		(at 168.402 195.326 0)
+		(effects
+			(font
+				(size 1.27 1.27)
+			)
+		)
 	)
 	(junction
@@
 			(project "l8-kicad"
 				(path "/09e08bdc-786f-4949-8afc-e02ddbe0502e/1f4251eb-3452-4303-bba0-dce7319e59b1"
-					(reference "D802")
+					(reference "D801")
 					(unit 1)
 				)
@@
 			)
 			(project "l8-kicad"
-				(path "/8d063f79-9282-4820-bcf4-1ff3c006cf08/ad2e8a4f-4087-4a5a-8ddd-b6c7bc1c0b58"
+				(path "/8d063f79-9282-4820-bcf4-1ff3c006cf08/afe0b366-72e8-4aeb-bdd6-ed92c2bd7364"
 					(reference "D802")
 					(unit 1)
@@
 			)
 			(project "l8-kicad"
-				(path "/8d063f79-9282-4820-bcf4-1ff3c006cf08/ad2e8a4f-4087-4a5a-8ddd-b6c7bc1c0b58"
+				(path "/8d063f79-9282-4820-bcf4-1ff3c006cf08/afe0b366-72e8-4aeb-bdd6-ed92c2bd7364"
 					(reference "F801")
 					(unit 1)
@@
 			)
 			(project "l8-kicad"
-				(path "/8d063f79-9282-4820-bcf4-1ff3c006cf08/ad2e8a4f-4087-4a5a-8ddd-b6c7bc1c0b58"
+				(path "/8d063f79-9282-4820-bcf4-1ff3c006cf08/afe0b366-72e8-4aeb-bdd6-ed92c2bd7364"
 					(reference "#PWR0801")
 					(unit 1)
@@
 			(project "l8-kicad"
 				(path "/09e08bdc-786f-4949-8afc-e02ddbe0502e/1f4251eb-3452-4303-bba0-dce7319e59b1"
-					(reference "R701")
+					(reference "R805")
 					(unit 1)
 				)
@@
 			)
 			(project "l8-kicad"
-				(path "/8d063f79-9282-4820-bcf4-1ff3c006cf08/ad2e8a4f-4087-4a5a-8ddd-b6c7bc1c0b58"
+				(path "/8d063f79-9282-4820-bcf4-1ff3c006cf08/afe0b366-72e8-4aeb-bdd6-ed92c2bd7364"
 					(reference "R701")
 					(unit 1)
@@
 			)
 			(project "l8-kicad"
-				(path "/8d063f79-9282-4820-bcf4-1ff3c006cf08/ad2e8a4f-4087-4a5a-8ddd-b6c7bc1c0b58"
+				(path "/8d063f79-9282-4820-bcf4-1ff3c006cf08/afe0b366-72e8-4aeb-bdd6-ed92c2bd7364"
 					(reference "#PWR0808")
 					(unit 1)
@@
 			)
 			(project "l8-kicad"
-				(path "/8d063f79-9282-4820-bcf4-1ff3c006cf08/ad2e8a4f-4087-4a5a-8ddd-b6c7bc1c0b58"
+				(path "/8d063f79-9282-4820-bcf4-1ff3c006cf08/afe0b366-72e8-4aeb-bdd6-ed92c2bd7364"
 					(reference "#PWR0802")
 					(unit 1)
@@
 			)
 			(project "l8-kicad"
-				(path "/8d063f79-9282-4820-bcf4-1ff3c006cf08/ad2e8a4f-4087-4a5a-8ddd-b6c7bc1c0b58"
+				(path "/8d063f79-9282-4820-bcf4-1ff3c006cf08/afe0b366-72e8-4aeb-bdd6-ed92c2bd7364"
 					(reference "R801")
 					(unit 1)
@@
 			)
 			(project "l8-kicad"
-				(path "/8d063f79-9282-4820-bcf4-1ff3c006cf08/ad2e8a4f-4087-4a5a-8ddd-b6c7bc1c0b58"
+				(path "/8d063f79-9282-4820-bcf4-1ff3c006cf08/afe0b366-72e8-4aeb-bdd6-ed92c2bd7364"
 					(reference "R802")
 					(unit 1)
@@
 			(project "l8-kicad"
 				(path "/09e08bdc-786f-4949-8afc-e02ddbe0502e/1f4251eb-3452-4303-bba0-dce7319e59b1"
-					(reference "R702")
+					(reference "R804")
 					(unit 1)
 				)
@@
 			)
 			(project "l8-kicad"
-				(path "/8d063f79-9282-4820-bcf4-1ff3c006cf08/ad2e8a4f-4087-4a5a-8ddd-b6c7bc1c0b58"
+				(path "/8d063f79-9282-4820-bcf4-1ff3c006cf08/afe0b366-72e8-4aeb-bdd6-ed92c2bd7364"
 					(reference "R702")
 					(unit 1)
@@
 			(project "l8-kicad"
 				(path "/09e08bdc-786f-4949-8afc-e02ddbe0502e/1f4251eb-3452-4303-bba0-dce7319e59b1"
-					(reference "D801")
+					(reference "D802")
 					(unit 1)
 				)
@@
 			)
 			(project "l8-kicad"
-				(path "/8d063f79-9282-4820-bcf4-1ff3c006cf08/ad2e8a4f-4087-4a5a-8ddd-b6c7bc1c0b58"
+				(path "/8d063f79-9282-4820-bcf4-1ff3c006cf08/afe0b366-72e8-4aeb-bdd6-ed92c2bd7364"
 					(reference "D801")
 					(unit 1)
@@
 			(project "l8-kicad"
 				(path "/09e08bdc-786f-4949-8afc-e02ddbe0502e/1f4251eb-3452-4303-bba0-dce7319e59b1"
-					(reference "#PWR0804")
+					(reference "#PWR0806")
 					(unit 1)
 				)
@@
 			)
 			(project "l8-kicad"
-				(path "/8d063f79-9282-4820-bcf4-1ff3c006cf08/ad2e8a4f-4087-4a5a-8ddd-b6c7bc1c0b58"
+				(path "/8d063f79-9282-4820-bcf4-1ff3c006cf08/afe0b366-72e8-4aeb-bdd6-ed92c2bd7364"
 					(reference "#PWR0804")
 					(unit 1)
@@
 			(project "l8-kicad"
 				(path "/09e08bdc-786f-4949-8afc-e02ddbe0502e/1f4251eb-3452-4303-bba0-dce7319e59b1"
-					(reference "#PWR0805")
+					(reference "#PWR0804")
 					(unit 1)
 				)
@@
 			)
 			(project "l8-kicad"
-				(path "/8d063f79-9282-4820-bcf4-1ff3c006cf08/ad2e8a4f-4087-4a5a-8ddd-b6c7bc1c0b58"
+				(path "/8d063f79-9282-4820-bcf4-1ff3c006cf08/afe0b366-72e8-4aeb-bdd6-ed92c2bd7364"
 					(reference "#PWR0805")
 					(unit 1)
@@
 			)
 			(project "l8-kicad"
-				(path "/8d063f79-9282-4820-bcf4-1ff3c006cf08/ad2e8a4f-4087-4a5a-8ddd-b6c7bc1c0b58"
+				(path "/8d063f79-9282-4820-bcf4-1ff3c006cf08/afe0b366-72e8-4aeb-bdd6-ed92c2bd7364"
 					(reference "R803")
 					(unit 1)
@@
 			)
 			(project "l8-kicad"
-				(path "/8d063f79-9282-4820-bcf4-1ff3c006cf08/ad2e8a4f-4087-4a5a-8ddd-b6c7bc1c0b58"
+				(path "/8d063f79-9282-4820-bcf4-1ff3c006cf08/afe0b366-72e8-4aeb-bdd6-ed92c2bd7364"
 					(reference "J801")
 					(unit 1)
@@
 			)
 			(project "l8-kicad"
-				(path "/8d063f79-9282-4820-bcf4-1ff3c006cf08/ad2e8a4f-4087-4a5a-8ddd-b6c7bc1c0b58"
+				(path "/8d063f79-9282-4820-bcf4-1ff3c006cf08/afe0b366-72e8-4aeb-bdd6-ed92c2bd7364"
 					(reference "#PWR0807")
 					(unit 1)
@@
 			(project "l8-kicad"
 				(path "/09e08bdc-786f-4949-8afc-e02ddbe0502e/1f4251eb-3452-4303-bba0-dce7319e59b1"
-					(reference "#PWR0806")
+					(reference "#PWR0805")
 					(unit 1)
 				)
@@
 			)
 			(project "l8-kicad"
-				(path "/8d063f79-9282-4820-bcf4-1ff3c006cf08/ad2e8a4f-4087-4a5a-8ddd-b6c7bc1c0b58"
+				(path "/8d063f79-9282-4820-bcf4-1ff3c006cf08/afe0b366-72e8-4aeb-bdd6-ed92c2bd7364"
 					(reference "#PWR0806")
 					(unit 1)
@@
 			)
 			(project "l8-kicad"
-				(path "/8d063f79-9282-4820-bcf4-1ff3c006cf08/ad2e8a4f-4087-4a5a-8ddd-b6c7bc1c0b58"
+				(path "/8d063f79-9282-4820-bcf4-1ff3c006cf08/afe0b366-72e8-4aeb-bdd6-ed92c2bd7364"
 					(reference "C801")
 					(unit 1)
@@
 			)
 			(project "l8-kicad"
-				(path "/8d063f79-9282-4820-bcf4-1ff3c006cf08/ad2e8a4f-4087-4a5a-8ddd-b6c7bc1c0b58"
+				(path "/8d063f79-9282-4820-bcf4-1ff3c006cf08/afe0b366-72e8-4aeb-bdd6-ed92c2bd7364"
 					(reference "#PWR0803")
 					(unit 1)

Commit message: x
Parts:
- R701: footprint Resistor_SMD:R_0603_1608Metric -> (none); LCSC C4190 -> (none)
- R702: footprint Resistor_SMD:R_0603_1608Metric -> (none); LCSC C25804 -> (none)
- R803: footprint PCM_JLCPCB:R_0603 -> (none); LCSC C23186 -> (none)
Changed lines of the file:
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@@
 			)
 		)
-		(property "Datasheet" "http://www.onsemi.com/pub_link/Collateral/NUP4202W1-D.PDF"
+		(property "Datasheet" ""
 			(at 95.25 133.35 90)
 			(effects
@@
 			)
 		)
-		(property "Footprint" "Resistor_SMD:R_0603_1608Metric"
+		(property "Footprint" ""
 			(at 160.528 133.35 90)
 			(effects
@@
 		)
 		(property "Description" "Resistor"
-			(at 158.75 133.35 0)
-			(effects
-				(font
-					(size 1.27 1.27)
-				)
-				(hide yes)
-			)
-		)
-		(property "LCSC" "C4190"
-			(at 158.75 133.35 0)
-			(effects
-				(font
-					(size 1.27 1.27)
-				)
-				(hide yes)
-			)
-		)
-		(property "Manufacturer" ""
-			(at 158.75 133.35 0)
-			(effects
-				(font
-					(size 1.27 1.27)
-				)
-				(hide yes)
-			)
-		)
-		(property "Part #" ""
-			(at 158.75 133.35 0)
-			(effects
-				(font
-					(size 1.27 1.27)
-				)
-				(hide yes)
-			)
-		)
-		(property "VEND" ""
-			(at 158.75 133.35 0)
-			(effects
-				(font
-					(size 1.27 1.27)
-				)
-				(hide yes)
-			)
-		)
-		(property "VEND#" ""
-			(at 158.75 133.35 0)
-			(effects
-				(font
-					(size 1.27 1.27)
-				)
-				(hide yes)
-			)
-		)
-		(property "Sim.Device" ""
-			(at 158.75 133.35 0)
-			(effects
-				(font
-					(size 1.27 1.27)
-				)
-				(hide yes)
-			)
-		)
-		(property "Sim.Pins" ""
-			(at 158.75 133.35 0)
-			(effects
-				(font
-					(size 1.27 1.27)
-				)
-				(hide yes)
-			)
-		)
-		(property "Silkscreen" ""
 			(at 158.75 133.35 0)
 			(effects
@@
 			)
 		)
-		(property "Footprint" "Resistor_SMD:R_0603_1608Metric"
-			(at 210.82 37.338 90)
-			(effects
-				(font
-					(size 1.524 1.524)
+		(property "Footprint" ""
+			(at 152.4 98.298 90)
+			(effects
+				(font
+					(size 1.27 1.27)
 				)
 				(hide yes)
@@
 		)
 		(property "Datasheet" "~"
-			(at 211.455 -52.07 0)
-			(effects
-				(font
-					(size 1.524 1.524)
+			(at 152.4 96.52 0)
+			(effects
+				(font
+					(size 1.27 1.27)
 				)
 				(hide yes)
@@
 		)
 		(property "Description" "Resistor"
-			(at 152.4 96.52 0)
-			(effects
-				(font
-					(size 1.27 1.27)
-				)
-				(hide yes)
-			)
-		)
-		(property "Part #" ""
-			(at 54.61 199.39 0)
-			(effects
-				(font
-					(size 1.27 1.27)
-				)
-				(hide yes)
-			)
-		)
-		(property "VEND" ""
-			(at 54.61 199.39 0)
-			(effects
-				(font
-					(size 1.27 1.27)
-				)
-				(hide yes)
-			)
-		)
-		(property "VEND#" ""
-			(at 54.61 199.39 0)
-			(effects
-				(font
-					(size 1.27 1.27)
-				)
-				(hide yes)
-			)
-		)
-		(property "Manufacturer" ""
-			(at 54.61 199.39 0)
-			(effects
-				(font
-					(size 1.27 1.27)
-				)
-				(hide yes)
-			)
-		)
-		(property "LCSC" "C25804"
-			(at 152.4 96.52 0)
-			(effects
-				(font
-					(size 1.27 1.27)
-				)
-				(hide yes)
-			)
-		)
-		(property "Sim.Device" ""
-			(at 152.4 96.52 0)
-			(effects
-				(font
-					(size 1.27 1.27)
-				)
-				(hide yes)
-			)
-		)
-		(property "Sim.Pins" ""
-			(at 152.4 96.52 0)
-			(effects
-				(font
-					(size 1.27 1.27)
-				)
-				(hide yes)
-			)
-		)
-		(property "Silkscreen" ""
 			(at 152.4 96.52 0)
 			(effects
@@
 		)
 		(property "Value" "+5V"
-			(at 142.24 67.3099 0)
-			(effects
-				(font
-					(size 1.27 1.27)
-				)
-				(justify left)
+			(at 139.7 63.5 0)
+			(effects
+				(font
+					(size 1.27 1.27)
+				)
 			)
 		)
@@
 			)
 		)
-		(property "Footprint" "PCM_JLCPCB:R_0603"
+		(property "Footprint" ""
 			(at 137.922 133.35 90)
 			(effects
@@
 			)
 		)
-		(property "Datasheet" "https://www.lcsc.com/datasheet/lcsc_datasheet_2206010116_UNI-ROYAL-Uniroyal-Elec-0603WAF5101T5E_C23186.pdf"
+		(property "Datasheet" "~"
 			(at 139.7 133.35 0)
 			(effects
@@
 			(effects
 				(font
-					(size 1.27 1.27)
-				)
-				(hide yes)
-			)
-		)
-		(property "LCSC" "C23186"
-			(at 139.7 133.35 90)
-			(effects
-				(font

Commit message: pdm sch drc clean
Parts:
- R701: value 2.2K -> 2.2kΩ; footprint (none) -> PCM_JLCPCB:R_0402; symbol Device:R -> dnt_global:Resistor_0402,2.2kΩ; Attrition Qty (none) -> 10; Category (none) -> Resistors,Chip Resistor - Surface Mount; Class (none) -> Basic Component; LCSC (none) -> C25879; Manufacturer (none) -> UNI-ROYAL(Uniroyal Elec); Minimum Qty (none) -> 20; Operating Temperature Range (none) -> -55°C~+155°C; Overload Voltage (Max) (none) -> 50V; Part (none) -> 0402WGF2201TCE; Power(Watts) (none) -> 62.5mW; Price (none) -> 0.004USD; Process (none) -> SMT; Resistance (none) -> 2.2kΩ; Stock (none) -> 1767502; Temperature Coefficient (none) -> ±100ppm/°C; Tolerance (none) -> ±1%; Type (none) -> Thick Film Resistors
- R702: footprint (none) -> PCM_JLCPCB:R_0402; symbol Device:R -> dnt_global:Resistor_0402,10kΩ; Attrition Qty (none) -> 10; Category (none) -> Resistors,Chip Resistor - Surface Mount; Class (none) -> Basic Component; LCSC (none) -> C25744; Manufacturer (none) -> UNI-ROYAL(Uniroyal Elec); Minimum Qty (none) -> 20; Operating Temperature Range (none) -> -55°C~+155°C; Overload Voltage (Max) (none) -> 50V; Part (none) -> 0402WGF1002TCE; Power(Watts) (none) -> 62.5mW; Price (none) -> 0.004USD; Process (none) -> SMT; Resistance (none) -> 10kΩ; Stock (none) -> 24372091; Temperature Coefficient (none) -> ±100ppm/°C; Tolerance (none) -> ±1%; Type (none) -> Thick Film Resistors
- R802: footprint PCM_JLCPCB:R_0603 -> PCM_JLCPCB:R_0402; symbol PCM_JLCPCB-Resistors:0603,5.1kΩ -> dnt_global:Resistor_0402,5.1kΩ; LCSC C23186 -> C25905; Overload Voltage (Max) 75V -> 50V; Part 0603WAF5101T5E -> 0402WGF5101TCE; Power(Watts) 100mW -> 62.5mW; Stock 9223405 -> 3534773
- R803: value 5.1K -> 5.1kΩ; footprint (none) -> PCM_JLCPCB:R_0402; symbol Device:R -> dnt_global:Resistor_0402,5.1kΩ; Attrition Qty (none) -> 10; Category (none) -> Resistors,Chip Resistor - Surface Mount; Class (none) -> Basic Component; LCSC (none) -> C25905; Manufacturer (none) -> UNI-ROYAL(Uniroyal Elec); Minimum Qty (none) -> 20; Operating Temperature Range (none) -> -55°C~+155°C; Overload Voltage (Max) (none) -> 50V; Part (none) -> 0402WGF5101TCE; Power(Watts) (none) -> 62.5mW; Price (none) -> 0.004USD; Process (none) -> SMT; Resistance (none) -> 5.1kΩ; Stock (none) -> 3534773; Temperature Coefficient (none) -> ±100ppm/°C; Tolerance (none) -> ±1%; Type (none) -> Thick Film Resistors

Commit message: lcd power switch-- add new accelerometer
Parts:
- renumbered D802 to D801, D801 to D802, R702 to R804, R701 to R805
Changed lines of the file:
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@@
 		(on_board yes)
 		(dnp no)
-		(property "Reference" "D802"
+		(property "Reference" "D?"
 			(at 103.632 132.1816 0)
 			(effects
@@
 				)
 			)
-			(project "l8-kicad"
-				(path "/8d063f79-9282-4820-bcf4-1ff3c006cf08/afe0b366-72e8-4aeb-bdd6-ed92c2bd7364"
-					(reference "D802")
+			(project "z9-console"
+				(path "/8d063f79-9282-4820-bcf4-1ff3c006cf08/ad2e8a4f-4087-4a5a-8ddd-b6c7bc1c0b58"
+					(reference "D?")
 					(unit 1)
 				)
@@
 		(dnp no)
 		(fields_autoplaced yes)
-		(property "Reference" "F801"
+		(property "Reference" "F?"
 			(at 77.47 90.17 90)
 			(effects
@@
 				)
 			)
-			(project "l8-kicad"
-				(path "/8d063f79-9282-4820-bcf4-1ff3c006cf08/afe0b366-72e8-4aeb-bdd6-ed92c2bd7364"
-					(reference "F801")
+			(project "z9-console"
+				(path "/8d063f79-9282-4820-bcf4-1ff3c006cf08/ad2e8a4f-4087-4a5a-8ddd-b6c7bc1c0b58"
+					(reference "F?")
 					(unit 1)
 				)
@@
 		(on_board yes)
 		(dnp no)
-		(property "Reference" "#PWR0801"
+		(property "Reference" "#PWR?"
 			(at 36.83 154.94 0)
 			(effects
@@
 				)
 			)
-			(project "l8-kicad"
-				(path "/8d063f79-9282-4820-bcf4-1ff3c006cf08/afe0b366-72e8-4aeb-bdd6-ed92c2bd7364"
-					(reference "#PWR0801")
+			(project "z9-console"
+				(path "/8d063f79-9282-4820-bcf4-1ff3c006cf08/ad2e8a4f-4087-4a5a-8ddd-b6c7bc1c0b58"
+					(reference "#PWR?")
 					(unit 1)
 				)
@@
 		(on_board yes)
 		(dnp no)
-		(property "Reference" "R701"
+		(property "Reference" "R?"
 			(at 156.972 133.35 0)
 			(effects
@@
 				)
 			)
-			(project "l8-kicad"
-				(path "/8d063f79-9282-4820-bcf4-1ff3c006cf08/afe0b366-72e8-4aeb-bdd6-ed92c2bd7364"
-					(reference "R701")
+			(project "z9-console"
+				(path "/8d063f79-9282-4820-bcf4-1ff3c006cf08/ad2e8a4f-4087-4a5a-8ddd-b6c7bc1c0b58"
+					(reference "R?")
 					(unit 1)
 				)
@@
 		(on_board yes)
 		(dnp no)
-		(property "Reference" "#PWR0808"
+		(property "Reference" "#PWR?"
 			(at 158.75 154.94 0)
 			(effects
@@
 				)
 			)
-			(project "l8-kicad"
-				(path "/8d063f79-9282-4820-bcf4-1ff3c006cf08/afe0b366-72e8-4aeb-bdd6-ed92c2bd7364"
-					(reference "#PWR0808")
+			(project "z9-console"
+				(path "/8d063f79-9282-4820-bcf4-1ff3c006cf08/ad2e8a4f-4087-4a5a-8ddd-b6c7bc1c0b58"
+					(reference "#PWR?")
 					(unit 1)
 				)
@@
 		(on_board yes)
 		(dnp no)
-		(property "Reference" "#PWR0802"
+		(property "Reference" "#PWR?"
 			(at 45.72 154.94 0)
 			(effects
@@
 				)
 			)
-			(project "l8-kicad"
-				(path "/8d063f79-9282-4820-bcf4-1ff3c006cf08/afe0b366-72e8-4aeb-bdd6-ed92c2bd7364"
-					(reference "#PWR0802")
+			(project "z9-console"
+				(path "/8d063f79-9282-4820-bcf4-1ff3c006cf08/ad2e8a4f-4087-4a5a-8ddd-b6c7bc1c0b58"
+					(reference "#PWR?")
 					(unit 1)
 				)
@@
 		(on_board yes)
 		(dnp no)
-		(property "Reference" "R801"
+		(property "Reference" "R?"
 			(at 34.798 146.05 90)
 			(effects
@@
 				)
 			)
-			(project "l8-kicad"
-				(path "/8d063f79-9282-4820-bcf4-1ff3c006cf08/afe0b366-72e8-4aeb-bdd6-ed92c2bd7364"
-					(reference "R801")
+			(project "z9-console"
+				(path "/8d063f79-9282-4820-bcf4-1ff3c006cf08/ad2e8a4f-4087-4a5a-8ddd-b6c7bc1c0b58"
+					(reference "R?")
 					(unit 1)
 				)
@@
 		(on_board yes)
 		(dnp no)
-		(property "Reference" "R802"
+		(property "Reference" "R?"
 			(at 131.318 133.35 0)
 			(effects
@@
 				)
 			)
-			(project "l8-kicad"
-				(path "/8d063f79-9282-4820-bcf4-1ff3c006cf08/afe0b366-72e8-4aeb-bdd6-ed92c2bd7364"
-					(reference "R802")
+			(project "z9-console"
+				(path "/8d063f79-9282-4820-bcf4-1ff3c006cf08/ad2e8a4f-4087-4a5a-8ddd-b6c7bc1c0b58"
+					(reference "R?")
 					(unit 1)
 				)
@@
 		(on_board yes)
 		(dnp no)
-		(property "Reference" "R702"
+		(property "Reference" "R?"
 			(at 152.4 94.488 90)
 			(effects
@@
 				)
 			)
-			(project "l8-kicad"
-				(path "/8d063f79-9282-4820-bcf4-1ff3c006cf08/afe0b366-72e8-4aeb-bdd6-ed92c2bd7364"
-					(reference "R702")
+			(project "z9-console"
+				(path "/8d063f79-9282-4820-bcf4-1ff3c006cf08/ad2e8a4f-4087-4a5a-8ddd-b6c7bc1c0b58"
+					(reference "R?")
 					(unit 1)
 				)
@@
 		(dnp no)
 		(fields_autoplaced yes)
-		(property "Reference" "D801"
+		(property "Reference" "D?"
 			(at 142.24 75.8824 0)
 			(effects
@@
 				)
 			)
-			(project "l8-kicad"
-				(path "/8d063f79-9282-4820-bcf4-1ff3c006cf08/afe0b366-72e8-4aeb-bdd6-ed92c2bd7364"
-					(reference "D801")
+			(project "z9-console"
+				(path "/8d063f79-9282-4820-bcf4-1ff3c006cf08/ad2e8a4f-4087-4a5a-8ddd-b6c7bc1c0b58"
+					(reference "D?")
 					(unit 1)
 				)
@@
 		(dnp no)
 		(fields_autoplaced yes)
-		(property "Reference" "#PWR0804"
+		(property "Reference" "#PWR?"
 			(at 139.7 72.39 0)
 			(effects
@@
 				)
 			)
-			(project "l8-kicad"
-				(path "/8d063f79-9282-4820-bcf4-1ff3c006cf08/afe0b366-72e8-4aeb-bdd6-ed92c2bd7364"
-					(reference "#PWR0804")
+			(project "z9-console"
+				(path "/8d063f79-9282-4820-bcf4-1ff3c006cf08/ad2e8a4f-4087-4a5a-8ddd-b6c7bc1c0b58"
+					(reference "#PWR?")
 					(unit 1)
 				)
@@
 		(on_board yes)
 		(dnp no)
-		(property "Reference" "#PWR0805"
+		(property "Reference" "#PWR?"
 			(at 95.25 154.94 0)
 			(effects
@@
 				)
 			)
-			(project "l8-kicad"
-				(path "/8d063f79-9282-4820-bcf4-1ff3c006cf08/afe0b366-72e8-4aeb-bdd6-ed92c2bd7364"
-					(reference "#PWR0805")
+			(project "z9-console"
+				(path "/8d063f79-9282-4820-bcf4-1ff3c006cf08/ad2e8a4f-4087-4a5a-8ddd-b6c7bc1c0b58"
+					(reference "#PWR?")
 					(unit 1)
 				)
@@
 		(on_board yes)
 		(dnp no)
-		(property "Reference" "R803"
+		(property "Reference" "R?"
 			(at 141.478 133.35 0)
 			(effects
@@
 				)
 			)
-			(project "l8-kicad"
-				(path "/8d063f79-9282-4820-bcf4-1ff3c006cf08/afe0b366-72e8-4aeb-bdd6-ed92c2bd7364"
-					(reference "R803")
+			(project "z9-console"
+				(path "/8d063f79-9282-4820-bcf4-1ff3c006cf08/ad2e8a4f-4087-4a5a-8ddd-b6c7bc1c0b58"
+					(reference "R?")
 					(unit 1)
 				)
@@
 		(dnp no)
 		(fields_autoplaced yes)
-		(property "Reference" "J801"
+		(property "Reference" "J?"
 			(at 53.34 88.9 0)
 			(effects
@@
 				)
 			)
-			(project "l8-kicad"
-				(path "/8d063f79-9282-4820-bcf4-1ff3c006cf08/afe0b366-72e8-4aeb-bdd6-ed92c2bd7364"
-					(reference "J801")
+			(project "z9-console"
+				(path "/8d063f79-9282-4820-bcf4-1ff3c006cf08/ad2e8a4f-4087-4a5a-8ddd-b6c7bc1c0b58"
+					(reference "J?")
 					(unit 1)
 				)
@@
 		(dnp no)
 		(fields_autoplaced yes)
-		(property "Reference" "#PWR0807"
+		(property "Reference" "#PWR?"
 			(at 139.7 161.29 0)
 			(effects
@@
 				)
 			)
-			(project "l8-kicad"
-				(path "/8d063f79-9282-4820-bcf4-1ff3c006cf08/afe0b366-72e8-4aeb-bdd6-ed92c2bd7364"
-					(reference "#PWR0807")
+			(project "z9-console"
+				(path "/8d063f79-9282-4820-bcf4-1ff3c006cf08/ad2e8a4f-4087-4a5a-8ddd-b6c7bc1c0b58"
+					(reference "#PWR?")
 					(unit 1)
 				)
@@
 		(dnp no)
 		(fields_autoplaced yes)
-		(property "Reference" "#PWR0806"
+		(property "Reference" "#PWR?"
 			(at 129.54 161.29 0)
 			(effects
@@
 				)
 			)
-			(project "l8-kicad"
-				(path "/8d063f79-9282-4820-bcf4-1ff3c006cf08/afe0b366-72e8-4aeb-bdd6-ed92c2bd7364"
-					(reference "#PWR0806")
+			(project "z9-console"
+				(path "/8d063f79-9282-4820-bcf4-1ff3c006cf08/ad2e8a4f-4087-4a5a-8ddd-b6c7bc1c0b58"
+					(reference "#PWR?")
 					(unit 1)
 				)
@@
 		(on_board yes)
 		(dnp no)
-		(property "Reference" "C801"
+		(property "Reference" "C?"
 			(at 46.99 146.05 90)
 			(effects
@@
 				)
 			)
-			(project "l8-kicad"
-				(path "/8d063f79-9282-4820-bcf4-1ff3c006cf08/afe0b366-72e8-4aeb-bdd6-ed92c2bd7364"
-					(reference "C801")
+			(project "z9-console"
+				(path "/8d063f79-9282-4820-bcf4-1ff3c006cf08/ad2e8a4f-4087-4a5a-8ddd-b6c7bc1c0b58"
+					(reference "C?")
 					(unit 1)
 				)
@@
 		(on_board yes)
 		(dnp no)
-		(property "Reference" "#PWR0803"
+		(property "Reference" "#PWR?"
 			(at 53.34 154.94 0)
 			(effects
@@
 				)
 			)
-			(project "l8-kicad"
-				(path "/8d063f79-9282-4820-bcf4-1ff3c006cf08/afe0b366-72e8-4aeb-bdd6-ed92c2bd7364"
-					(reference "#PWR0803")
+			(project "z9-console"
+				(path "/8d063f79-9282-4820-bcf4-1ff3c006cf08/ad2e8a4f-4087-4a5a-8ddd-b6c7bc1c0b58"
+					(reference "#PWR?")
 					(unit 1)
 				)
