File: z9-shared/shared_usbc.kicad_sch (KiCad schematic)
At the start: 10 parts, among them J801 USB_C_Receptacle_USB2.0_16P

Commit message: change MEMS device
Parts:
- renumbered C801 to C930, D801 to D916, D802 to D917, F801 to F904, J801 to J910, R801 to R929, R802 to R930, R803 to R931, R804 to R932, R805 to R933
Changed lines of the file:
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@@
 		(on_board yes)
 		(dnp no)
-		(property "Reference" "D?"
+		(property "Reference" "D916"
 			(at 103.632 132.1816 0)
 			(effects
@@
 			(project "z9-console"
 				(path "/8d063f79-9282-4820-bcf4-1ff3c006cf08/ad2e8a4f-4087-4a5a-8ddd-b6c7bc1c0b58"
-					(reference "D?")
+					(reference "D916")
 					(unit 1)
 				)
@@
 		(dnp no)
 		(fields_autoplaced yes)
-		(property "Reference" "F?"
+		(property "Reference" "F904"
 			(at 77.47 90.17 90)
 			(effects
@@
 			(project "z9-console"
 				(path "/8d063f79-9282-4820-bcf4-1ff3c006cf08/ad2e8a4f-4087-4a5a-8ddd-b6c7bc1c0b58"
-					(reference "F?")
+					(reference "F904")
 					(unit 1)
 				)
@@
 		(on_board yes)
 		(dnp no)
-		(property "Reference" "#PWR?"
+		(property "Reference" "#PWR0949"
 			(at 36.83 154.94 0)
 			(effects
@@
 			(project "z9-console"
 				(path "/8d063f79-9282-4820-bcf4-1ff3c006cf08/ad2e8a4f-4087-4a5a-8ddd-b6c7bc1c0b58"
-					(reference "#PWR?")
+					(reference "#PWR0949")
 					(unit 1)
 				)
@@
 		(on_board yes)
 		(dnp no)
-		(property "Reference" "R?"
+		(property "Reference" "R933"
 			(at 156.972 133.35 0)
 			(effects
@@
 			(project "z9-console"
 				(path "/8d063f79-9282-4820-bcf4-1ff3c006cf08/ad2e8a4f-4087-4a5a-8ddd-b6c7bc1c0b58"
-					(reference "R?")
+					(reference "R933")
 					(unit 1)
 				)
@@
 		(on_board yes)
 		(dnp no)
-		(property "Reference" "#PWR?"
+		(property "Reference" "#PWR0956"
 			(at 158.75 154.94 0)
 			(effects
@@
 			(project "z9-console"
 				(path "/8d063f79-9282-4820-bcf4-1ff3c006cf08/ad2e8a4f-4087-4a5a-8ddd-b6c7bc1c0b58"
-					(reference "#PWR?")
+					(reference "#PWR0956")
 					(unit 1)
 				)
@@
 		(on_board yes)
 		(dnp no)
-		(property "Reference" "#PWR?"
+		(property "Reference" "#PWR0950"
 			(at 45.72 154.94 0)
 			(effects
@@
 			(project "z9-console"
 				(path "/8d063f79-9282-4820-bcf4-1ff3c006cf08/ad2e8a4f-4087-4a5a-8ddd-b6c7bc1c0b58"
-					(reference "#PWR?")
+					(reference "#PWR0950")
 					(unit 1)
 				)
@@
 		(on_board yes)
 		(dnp no)
-		(property "Reference" "R?"
+		(property "Reference" "R929"
 			(at 34.798 146.05 90)
 			(effects
@@
 			(project "z9-console"
 				(path "/8d063f79-9282-4820-bcf4-1ff3c006cf08/ad2e8a4f-4087-4a5a-8ddd-b6c7bc1c0b58"
-					(reference "R?")
+					(reference "R929")
 					(unit 1)
 				)
@@
 		(on_board yes)
 		(dnp no)
-		(property "Reference" "R?"
+		(property "Reference" "R930"
 			(at 131.318 133.35 0)
 			(effects
@@
 			(project "z9-console"
 				(path "/8d063f79-9282-4820-bcf4-1ff3c006cf08/ad2e8a4f-4087-4a5a-8ddd-b6c7bc1c0b58"
-					(reference "R?")
+					(reference "R930")
 					(unit 1)
 				)
@@
 		(on_board yes)
 		(dnp no)
-		(property "Reference" "R?"
+		(property "Reference" "R932"
 			(at 152.4 94.488 90)
 			(effects
@@
 			(project "z9-console"
 				(path "/8d063f79-9282-4820-bcf4-1ff3c006cf08/ad2e8a4f-4087-4a5a-8ddd-b6c7bc1c0b58"
-					(reference "R?")
+					(reference "R932")
 					(unit 1)
 				)
@@
 		(dnp no)
 		(fields_autoplaced yes)
-		(property "Reference" "D?"
+		(property "Reference" "D917"
 			(at 142.24 75.8824 0)
 			(effects
@@
 			(project "z9-console"
 				(path "/8d063f79-9282-4820-bcf4-1ff3c006cf08/ad2e8a4f-4087-4a5a-8ddd-b6c7bc1c0b58"
-					(reference "D?")
+					(reference "D917")
 					(unit 1)
 				)
@@
 		(dnp no)
 		(fields_autoplaced yes)
-		(property "Reference" "#PWR?"
+		(property "Reference" "#PWR0954"
 			(at 139.7 72.39 0)
 			(effects
@@
 			(project "z9-console"
 				(path "/8d063f79-9282-4820-bcf4-1ff3c006cf08/ad2e8a4f-4087-4a5a-8ddd-b6c7bc1c0b58"
-					(reference "#PWR?")
+					(reference "#PWR0954")
 					(unit 1)
 				)
@@
 		(on_board yes)
 		(dnp no)
-		(property "Reference" "#PWR?"
+		(property "Reference" "#PWR0952"
 			(at 95.25 154.94 0)
 			(effects
@@
 			(project "z9-console"
 				(path "/8d063f79-9282-4820-bcf4-1ff3c006cf08/ad2e8a4f-4087-4a5a-8ddd-b6c7bc1c0b58"
-					(reference "#PWR?")
+					(reference "#PWR0952")
 					(unit 1)
 				)
@@
 		(on_board yes)
 		(dnp no)
-		(property "Reference" "R?"
+		(property "Reference" "R931"
 			(at 141.478 133.35 0)
 			(effects
@@
 			(project "z9-console"
 				(path "/8d063f79-9282-4820-bcf4-1ff3c006cf08/ad2e8a4f-4087-4a5a-8ddd-b6c7bc1c0b58"
-					(reference "R?")
+					(reference "R931")
 					(unit 1)
 				)
@@
 		(dnp no)
 		(fields_autoplaced yes)
-		(property "Reference" "J?"
+		(property "Reference" "J910"
 			(at 53.34 88.9 0)
 			(effects
@@
 			(project "z9-console"
 				(path "/8d063f79-9282-4820-bcf4-1ff3c006cf08/ad2e8a4f-4087-4a5a-8ddd-b6c7bc1c0b58"
-					(reference "J?")
+					(reference "J910")
 					(unit 1)
 				)
@@
 		(dnp no)
 		(fields_autoplaced yes)
-		(property "Reference" "#PWR?"
+		(property "Reference" "#PWR0955"
 			(at 139.7 161.29 0)
 			(effects
@@
 			(project "z9-console"
 				(path "/8d063f79-9282-4820-bcf4-1ff3c006cf08/ad2e8a4f-4087-4a5a-8ddd-b6c7bc1c0b58"
-					(reference "#PWR?")
+					(reference "#PWR0955")
 					(unit 1)
 				)
@@
 		(dnp no)
 		(fields_autoplaced yes)
-		(property "Reference" "#PWR?"
+		(property "Reference" "#PWR0953"
 			(at 129.54 161.29 0)
 			(effects
@@
 			(project "z9-console"
 				(path "/8d063f79-9282-4820-bcf4-1ff3c006cf08/ad2e8a4f-4087-4a5a-8ddd-b6c7bc1c0b58"
-					(reference "#PWR?")
+					(reference "#PWR0953")
 					(unit 1)
 				)
@@
 		(on_board yes)
 		(dnp no)
-		(property "Reference" "C?"
+		(property "Reference" "C930"
 			(at 46.99 146.05 90)
 			(effects
@@
 			(project "z9-console"
 				(path "/8d063f79-9282-4820-bcf4-1ff3c006cf08/ad2e8a4f-4087-4a5a-8ddd-b6c7bc1c0b58"
-					(reference "C?")
+					(reference "C930")
 					(unit 1)
 				)
@@
 		(on_board yes)
 		(dnp no)
-		(property "Reference" "#PWR?"
+		(property "Reference" "#PWR0951"
 			(at 53.34 154.94 0)
 			(effects
@@
 			(project "z9-console"
 				(path "/8d063f79-9282-4820-bcf4-1ff3c006cf08/ad2e8a4f-4087-4a5a-8ddd-b6c7bc1c0b58"
-					(reference "#PWR?")
+					(reference "#PWR0951")
 					(unit 1)
 				)

Commit message: cleanup - change fus as test to shorten vale
Parts:
- renumbered C930 to C801, D916 to D801, D917 to D802, F904 to F801, J910 to J801, R929 to R801, R930 to R802, R931 to R803, R932 to R804, R933 to R805
Changed lines of the file:
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@@
 		(on_board yes)
 		(dnp no)
-		(property "Reference" "D916"
+		(property "Reference" "D?"
 			(at 103.632 132.1816 0)
 			(effects
@@
 				)
 			)
-			(project "z9-console"
-				(path "/8d063f79-9282-4820-bcf4-1ff3c006cf08/ad2e8a4f-4087-4a5a-8ddd-b6c7bc1c0b58"
-					(reference "D916")
+			(project "z9-pdm"
+				(path "/8d063f79-9282-4820-bcf4-1ff3c006cf08/afe0b366-72e8-4aeb-bdd6-ed92c2bd7364"
+					(reference "D?")
 					(unit 1)
 				)
@@
 		(dnp no)
 		(fields_autoplaced yes)
-		(property "Reference" "F904"
+		(property "Reference" "F?"
 			(at 77.47 90.17 90)
 			(effects
@@
 				)
 			)
-			(project "z9-console"
-				(path "/8d063f79-9282-4820-bcf4-1ff3c006cf08/ad2e8a4f-4087-4a5a-8ddd-b6c7bc1c0b58"
-					(reference "F904")
+			(project "z9-pdm"
+				(path "/8d063f79-9282-4820-bcf4-1ff3c006cf08/afe0b366-72e8-4aeb-bdd6-ed92c2bd7364"
+					(reference "F?")
 					(unit 1)
 				)
@@
 		(on_board yes)
 		(dnp no)
-		(property "Reference" "#PWR0949"
+		(property "Reference" "#PWR?"
 			(at 36.83 154.94 0)
 			(effects
@@
 				)
 			)
-			(project "z9-console"
-				(path "/8d063f79-9282-4820-bcf4-1ff3c006cf08/ad2e8a4f-4087-4a5a-8ddd-b6c7bc1c0b58"
-					(reference "#PWR0949")
+			(project "z9-pdm"
+				(path "/8d063f79-9282-4820-bcf4-1ff3c006cf08/afe0b366-72e8-4aeb-bdd6-ed92c2bd7364"
+					(reference "#PWR?")
 					(unit 1)
 				)
@@
 		(on_board yes)
 		(dnp no)
-		(property "Reference" "R933"
+		(property "Reference" "R?"
 			(at 156.972 133.35 0)
 			(effects
@@
 				)
 			)
-			(project "z9-console"
-				(path "/8d063f79-9282-4820-bcf4-1ff3c006cf08/ad2e8a4f-4087-4a5a-8ddd-b6c7bc1c0b58"
-					(reference "R933")
+			(project "z9-pdm"
+				(path "/8d063f79-9282-4820-bcf4-1ff3c006cf08/afe0b366-72e8-4aeb-bdd6-ed92c2bd7364"
+					(reference "R?")
 					(unit 1)
 				)
@@
 		(on_board yes)
 		(dnp no)
-		(property "Reference" "#PWR0956"
+		(property "Reference" "#PWR?"
 			(at 158.75 154.94 0)
 			(effects
@@
 				)
 			)
-			(project "z9-console"
-				(path "/8d063f79-9282-4820-bcf4-1ff3c006cf08/ad2e8a4f-4087-4a5a-8ddd-b6c7bc1c0b58"
-					(reference "#PWR0956")
+			(project "z9-pdm"
+				(path "/8d063f79-9282-4820-bcf4-1ff3c006cf08/afe0b366-72e8-4aeb-bdd6-ed92c2bd7364"
+					(reference "#PWR?")
 					(unit 1)
 				)
@@
 		(on_board yes)
 		(dnp no)
-		(property "Reference" "#PWR0950"
+		(property "Reference" "#PWR?"
 			(at 45.72 154.94 0)
 			(effects
@@
 				)
 			)
-			(project "z9-console"
-				(path "/8d063f79-9282-4820-bcf4-1ff3c006cf08/ad2e8a4f-4087-4a5a-8ddd-b6c7bc1c0b58"
-					(reference "#PWR0950")
+			(project "z9-pdm"
+				(path "/8d063f79-9282-4820-bcf4-1ff3c006cf08/afe0b366-72e8-4aeb-bdd6-ed92c2bd7364"
+					(reference "#PWR?")
 					(unit 1)
 				)
@@
 		(on_board yes)
 		(dnp no)
-		(property "Reference" "R929"
+		(property "Reference" "R?"
 			(at 34.798 146.05 90)
 			(effects
@@
 				)
 			)
-			(project "z9-console"
-				(path "/8d063f79-9282-4820-bcf4-1ff3c006cf08/ad2e8a4f-4087-4a5a-8ddd-b6c7bc1c0b58"
-					(reference "R929")
+			(project "z9-pdm"
+				(path "/8d063f79-9282-4820-bcf4-1ff3c006cf08/afe0b366-72e8-4aeb-bdd6-ed92c2bd7364"
+					(reference "R?")
 					(unit 1)
 				)
@@
 		(on_board yes)
 		(dnp no)
-		(property "Reference" "R930"
+		(property "Reference" "R?"
 			(at 131.318 133.35 0)
 			(effects
@@
 				)
 			)
-			(project "z9-console"
-				(path "/8d063f79-9282-4820-bcf4-1ff3c006cf08/ad2e8a4f-4087-4a5a-8ddd-b6c7bc1c0b58"
-					(reference "R930")
+			(project "z9-pdm"
+				(path "/8d063f79-9282-4820-bcf4-1ff3c006cf08/afe0b366-72e8-4aeb-bdd6-ed92c2bd7364"
+					(reference "R?")
 					(unit 1)
 				)
@@
 		(on_board yes)
 		(dnp no)
-		(property "Reference" "R932"
+		(property "Reference" "R?"
 			(at 152.4 94.488 90)
 			(effects
@@
 				)
 			)
-			(project "z9-console"
-				(path "/8d063f79-9282-4820-bcf4-1ff3c006cf08/ad2e8a4f-4087-4a5a-8ddd-b6c7bc1c0b58"
-					(reference "R932")
+			(project "z9-pdm"
+				(path "/8d063f79-9282-4820-bcf4-1ff3c006cf08/afe0b366-72e8-4aeb-bdd6-ed92c2bd7364"
+					(reference "R?")
 					(unit 1)
 				)
@@
 		(dnp no)
 		(fields_autoplaced yes)
-		(property "Reference" "D917"
+		(property "Reference" "D?"
 			(at 142.24 75.8824 0)
 			(effects
@@
 				)
 			)
-			(project "z9-console"
-				(path "/8d063f79-9282-4820-bcf4-1ff3c006cf08/ad2e8a4f-4087-4a5a-8ddd-b6c7bc1c0b58"
-					(reference "D917")
+			(project "z9-pdm"
+				(path "/8d063f79-9282-4820-bcf4-1ff3c006cf08/afe0b366-72e8-4aeb-bdd6-ed92c2bd7364"
+					(reference "D?")
 					(unit 1)
 				)
@@
 		(dnp no)
 		(fields_autoplaced yes)
-		(property "Reference" "#PWR0954"
+		(property "Reference" "#PWR?"
 			(at 139.7 72.39 0)
 			(effects
@@
 				)
 			)
-			(project "z9-console"
-				(path "/8d063f79-9282-4820-bcf4-1ff3c006cf08/ad2e8a4f-4087-4a5a-8ddd-b6c7bc1c0b58"
-					(reference "#PWR0954")
+			(project "z9-pdm"
+				(path "/8d063f79-9282-4820-bcf4-1ff3c006cf08/afe0b366-72e8-4aeb-bdd6-ed92c2bd7364"
+					(reference "#PWR?")
 					(unit 1)
 				)
@@
 		(on_board yes)
 		(dnp no)
-		(property "Reference" "#PWR0952"
+		(property "Reference" "#PWR?"
 			(at 95.25 154.94 0)
 			(effects
@@
 				)
 			)
-			(project "z9-console"
-				(path "/8d063f79-9282-4820-bcf4-1ff3c006cf08/ad2e8a4f-4087-4a5a-8ddd-b6c7bc1c0b58"
-					(reference "#PWR0952")
+			(project "z9-pdm"
+				(path "/8d063f79-9282-4820-bcf4-1ff3c006cf08/afe0b366-72e8-4aeb-bdd6-ed92c2bd7364"
+					(reference "#PWR?")
 					(unit 1)
 				)
@@
 		(on_board yes)
 		(dnp no)
-		(property "Reference" "R931"
+		(property "Reference" "R?"
 			(at 141.478 133.35 0)
 			(effects
@@
 				)
 			)
-			(project "z9-console"
-				(path "/8d063f79-9282-4820-bcf4-1ff3c006cf08/ad2e8a4f-4087-4a5a-8ddd-b6c7bc1c0b58"
-					(reference "R931")
+			(project "z9-pdm"
+				(path "/8d063f79-9282-4820-bcf4-1ff3c006cf08/afe0b366-72e8-4aeb-bdd6-ed92c2bd7364"
+					(reference "R?")
 					(unit 1)
 				)
@@
 		(dnp no)
 		(fields_autoplaced yes)
-		(property "Reference" "J910"
+		(property "Reference" "J?"
 			(at 53.34 88.9 0)
 			(effects
@@
 				)
 			)
-			(project "z9-console"
-				(path "/8d063f79-9282-4820-bcf4-1ff3c006cf08/ad2e8a4f-4087-4a5a-8ddd-b6c7bc1c0b58"
-					(reference "J910")
+			(project "z9-pdm"
+				(path "/8d063f79-9282-4820-bcf4-1ff3c006cf08/afe0b366-72e8-4aeb-bdd6-ed92c2bd7364"
+					(reference "J?")
 					(unit 1)
 				)
@@
 		(dnp no)
 		(fields_autoplaced yes)
-		(property "Reference" "#PWR0955"
+		(property "Reference" "#PWR?"
 			(at 139.7 161.29 0)
 			(effects
@@
 				)
 			)
-			(project "z9-console"
-				(path "/8d063f79-9282-4820-bcf4-1ff3c006cf08/ad2e8a4f-4087-4a5a-8ddd-b6c7bc1c0b58"
-					(reference "#PWR0955")
+			(project "z9-pdm"
+				(path "/8d063f79-9282-4820-bcf4-1ff3c006cf08/afe0b366-72e8-4aeb-bdd6-ed92c2bd7364"
+					(reference "#PWR?")
 					(unit 1)
 				)
@@
 		(dnp no)
 		(fields_autoplaced yes)
-		(property "Reference" "#PWR0953"
+		(property "Reference" "#PWR?"
 			(at 129.54 161.29 0)
 			(effects
@@
 				)
 			)
-			(project "z9-console"
-				(path "/8d063f79-9282-4820-bcf4-1ff3c006cf08/ad2e8a4f-4087-4a5a-8ddd-b6c7bc1c0b58"
-					(reference "#PWR0953")
+			(project "z9-pdm"
+				(path "/8d063f79-9282-4820-bcf4-1ff3c006cf08/afe0b366-72e8-4aeb-bdd6-ed92c2bd7364"
+					(reference "#PWR?")
 					(unit 1)
 				)
@@
 		(on_board yes)
 		(dnp no)
-		(property "Reference" "C930"
+		(property "Reference" "C?"
 			(at 46.99 146.05 90)
 			(effects
@@
 				)
 			)
-			(project "z9-console"
-				(path "/8d063f79-9282-4820-bcf4-1ff3c006cf08/ad2e8a4f-4087-4a5a-8ddd-b6c7bc1c0b58"
-					(reference "C930")
+			(project "z9-pdm"
+				(path "/8d063f79-9282-4820-bcf4-1ff3c006cf08/afe0b366-72e8-4aeb-bdd6-ed92c2bd7364"
+					(reference "C?")
 					(unit 1)
 				)
@@
 		(on_board yes)
 		(dnp no)
-		(property "Reference" "#PWR0951"
+		(property "Reference" "#PWR?"
 			(at 53.34 154.94 0)
 			(effects
@@
 				)
 			)
-			(project "z9-console"
-				(path "/8d063f79-9282-4820-bcf4-1ff3c006cf08/ad2e8a4f-4087-4a5a-8ddd-b6c7bc1c0b58"
-					(reference "#PWR0951")
+			(project "z9-pdm"
+				(path "/8d063f79-9282-4820-bcf4-1ff3c006cf08/afe0b366-72e8-4aeb-bdd6-ed92c2bd7364"
+					(reference "#PWR?")
 					(unit 1)
 				)

Commit message: reset shared chematics to correct series
Changed lines of the file:
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@@
 	(text "800 series"
 		(exclude_from_sim no)
-		(at 168.402 195.326 0)
+		(at 276.606 163.83 0)
 		(effects
 			(font
@@
 		(on_board yes)
 		(dnp no)
-		(property "Reference" "D?"
+		(property "Reference" "D801"
 			(at 103.632 132.1816 0)
 			(effects
@@
 		(dnp no)
 		(fields_autoplaced yes)
-		(property "Reference" "F?"
+		(property "Reference" "F801"
 			(at 77.47 90.17 90)
 			(effects
@@
 		(on_board yes)
 		(dnp no)
-		(property "Reference" "#PWR?"
+		(property "Reference" "#PWR0801"
 			(at 36.83 154.94 0)
 			(effects
@@
 		(on_board yes)
 		(dnp no)
-		(property "Reference" "R?"
+		(property "Reference" "R805"
 			(at 156.972 133.35 0)
 			(effects
@@
 		(on_board yes)
 		(dnp no)
-		(property "Reference" "#PWR?"
+		(property "Reference" "#PWR0808"
 			(at 158.75 154.94 0)
 			(effects
@@
 		(on_board yes)
 		(dnp no)
-		(property "Reference" "#PWR?"
+		(property "Reference" "#PWR0802"
 			(at 45.72 154.94 0)
 			(effects
@@
 		(on_board yes)
 		(dnp no)
-		(property "Reference" "R?"
+		(property "Reference" "R801"
 			(at 34.798 146.05 90)
 			(effects
@@
 		(on_board yes)
 		(dnp no)
-		(property "Reference" "R?"
+		(property "Reference" "R802"
 			(at 131.318 133.35 0)
 			(effects
@@
 		(on_board yes)
 		(dnp no)
-		(property "Reference" "R?"
+		(property "Reference" "R804"
 			(at 152.4 94.488 90)
 			(effects
@@
 		(dnp no)
 		(fields_autoplaced yes)
-		(property "Reference" "D?"
+		(property "Reference" "D802"
 			(at 142.24 75.8824 0)
 			(effects
@@
 		(dnp no)
 		(fields_autoplaced yes)
-		(property "Reference" "#PWR?"
+		(property "Reference" "#PWR0806"
 			(at 139.7 72.39 0)
 			(effects
@@
 		(on_board yes)
 		(dnp no)
-		(property "Reference" "#PWR?"
+		(property "Reference" "#PWR0804"
 			(at 95.25 154.94 0)
 			(effects
@@
 		(on_board yes)
 		(dnp no)
-		(property "Reference" "R?"
+		(property "Reference" "R803"
 			(at 141.478 133.35 0)
 			(effects
@@
 		(dnp no)
 		(fields_autoplaced yes)
-		(property "Reference" "J?"
+		(property "Reference" "J801"
 			(at 53.34 88.9 0)
 			(effects
@@
 		(dnp no)
 		(fields_autoplaced yes)
-		(property "Reference" "#PWR?"
+		(property "Reference" "#PWR0807"
 			(at 139.7 161.29 0)
 			(effects
@@
 		(dnp no)
 		(fields_autoplaced yes)
-		(property "Reference" "#PWR?"
+		(property "Reference" "#PWR0805"
 			(at 129.54 161.29 0)
 			(effects
@@
 		(on_board yes)
 		(dnp no)
-		(property "Reference" "C?"
+		(property "Reference" "C801"
 			(at 46.99 146.05 90)
 			(effects
@@
 		(on_board yes)
 		(dnp no)
-		(property "Reference" "#PWR?"
+		(property "Reference" "#PWR0803"
 			(at 53.34 154.94 0)
 			(effects
