File: z9-shared/shared_usbc.kicad_sch (KiCad schematic)
At the start: 10 parts, among them J801 USB_C_Receptacle_USB2.0_16P

Commit message: lcsc changes done - export for prod
Parts:
- R804: footprint PCM_JLCPCB:R_0402 -> dnt:R_0402_1005Metric; symbol dnt_global:Resistor_0402,10kΩ -> dnt_global:0402,10kΩ
Other:
- moved on the sheet: C801, D801, D802, F801, J801, R801, R802, R803, R804, R805

Commit message: more change - generarte jlc
Parts:
- D801: JLCPCB Rotation Offset 90 -> (none)
- R805: value 2.2kΩ -> 2.2k
Changed lines of the file:
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@@
 			)
 		)
-		(property "JLCPCB Rotation Offset" "90"
+		(property "JLCPCB Rotation Offset" ""
 			(at 120.65 115.57 0)
 			(effects
@@
 			)
 		)
-		(property "Value" "2.2kΩ"
+		(property "Value" "2.2k"
 			(at 184.15 115.57 90)
 			(do_not_autoplace yes)
