File: z9-shared/shared_usbc.kicad_sch (KiCad schematic)
At the start: 10 parts, among them J801 USB_C_Receptacle_USB2.0_16P

Commit message: sheet updates
Other:
- company: (none) -> Zero9 -  0-9.au
- title: l8 -> (none)
Changed lines of the file:
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@@
 	(paper "A4")
 	(title_block
-		(title "l8")
+		(company "Zero9 -  0-9.au")
+		(comment 1 "Some schematic is shared ")
 	)
 	(text "800 series"
