File: l8-harness/l8-harness.kicad_sch (KiCad schematic)
At the start: 27 parts, among them J1 Conn_01x06_Pin, J10 Conn_01x12_Socket, J11 Conn_01x12_Socket, J12 Conn_01x12_Pin, J2 Conn_01x06_Socket, J3 Conn_01x06_Socket, J4 Conn_01x06_Pin, J5 Conn_01x14_Pin, J6 Conn_01x21_Pin, J7 Conn_01x21_Socket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

Commit message: harness clean
Connections:
- net at F3.1, J4.1 (Pin_1): no longer F3.2
- net at BT1.2 (-), J9.1 (Pin_1), M1.2 (-): no longer F2.2, J8.1 (Pin_1)
- new net: F2.2, J8.1 (Pin_1)
Other:
- note added: "z9-pdm-901"
- note removed: "SCS-200"
Changed lines of the file:
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@@
 		)
 	)
-	(text "SCS-200"
+	(text "z9-pdm-901"
 		(exclude_from_sim no)
-		(at 285.496 202.184 0)
+		(at 305.816 152.654 90)
 		(effects
 			(font
@@
 	)
 	(junction
-		(at 259.08 111.76)
-		(diameter 0)
-		(color 0 0 0 0)
-	)
-	(junction
 		(at 30.48 49.53)
 		(diameter 0)
@@
 	)
 	(junction
-		(at 259.08 123.19)
-		(diameter 0)
-		(color 0 0 0 0)
-	)
-	(junction
 		(at 330.2 144.78)
 		(diameter 0)
@@
 	)
 	(junction
-		(at 242.57 115.57)
-		(diameter 0)
-		(color 0 0 0 0)
-	)
-	(junction
 		(at 330.2 74.93)
 		(diameter 0)
@@
 	)
 	(junction
-		(at 250.19 115.57)
-		(diameter 0)
-		(color 0 0 0 0)
-	)
-	(junction
 		(at 242.57 255.27)
 		(diameter 0)
@@
 	(wire
 		(pts
-			(xy 250.19 115.57) (xy 242.57 115.57)
-		)
-		(stroke
-			(width 0)
-			(type default)
-		)
-	)
-	(wire
-		(pts
 			(xy 330.2 187.96) (xy 378.46 187.96)
 		)
@@
 	(wire
 		(pts
-			(xy 256.54 115.57) (xy 250.19 115.57)
-		)
-		(stroke
-			(width 0)
-			(type default)
-		)
-	)
-	(wire
-		(pts
 			(xy 314.96 77.47) (xy 351.79 77.47)
 		)
@@
 	(wire
 		(pts
-			(xy 259.08 111.76) (xy 259.08 123.19)
-		)
-		(stroke
-			(width 0)
-			(type default)
-		)
-	)
-	(wire
-		(pts
 			(xy 236.22 212.09) (xy 240.03 212.09)
 		)
@@
 	(wire
 		(pts
+			(xy 250.19 115.57) (xy 256.54 115.57)
+		)
+		(stroke
+			(width 0)
+			(type default)
+		)
+	)
+	(wire
+		(pts
 			(xy 314.96 87.63) (xy 330.2 87.63)
 		)
@@
 			(type default)
 		)
-	)
-	(wire
-		(pts
-			(xy 259.08 111.76) (xy 259.08 113.03)
-		)
-		(stroke
-			(width 0.6096)
-			(type default)
-		)
