File: z9-console/stm32.kicad_sch (KiCad schematic)
At the start: 75 parts, among them J6 ST_STDC14 - SAMTEC_FTSH-107-0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, J7 TC2070 - TAG Connect, SW2 SW_Push, SW3 SW_Push, U8 STM32F427V_G-I_Tx, X2 8MHz 20pF

Commit message: remove bogus fields
Parts:
- C16, X2: PageName stm32f407_board -> (none)
Changed lines of the file:
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@@
 			)
 		)
-		(property "PageName" ""
-			(at 153.035 -129.54 0)
-			(effects
-				(font
-					(size 1.524 1.524)
-				)
-				(hide yes)
-			)
-		)
 		(property "Part #" ""
 			(at 207.01 229.87 0)
@@
 			)
 		)
-		(property "PageName" "stm32f407_board"
-			(at 215.265 -33.02 0)
-			(effects
-				(font
-					(size 1.524 1.524)
-				)
-				(hide yes)
-			)
-		)
 		(property "LCSC" "C115962"
 			(at 203.2 255.27 0)
@@
 			)
 		)
-		(property "PageName" "stm32f407_board"
-			(at -17.145 355.6 0)
-			(effects
-				(font
-					(size 1.524 1.524)
-				)
-				(hide yes)
-			)
-		)
 		(property "Part #" "GRM188R6YA225KA12D"
 			(at 15.24 80.01 0)
@@
 			)
 		)
-		(property "PageName" ""
-			(at -17.145 347.98 0)
-			(effects
-				(font
-					(size 1.524 1.524)
-				)
-				(hide yes)
-			)
-		)
 		(property "LCSC" "C23630"
 			(at 123.19 222.25 90)
@@
 			)
 		)
-		(property "PageName" ""
-			(at 194.945 541.02 0)
-			(effects
-				(font
-					(size 1.524 1.524)
-				)
-				(hide yes)
-			)
-		)
 		(property "Part #" "CL10C180JB8NNNC"
 			(at 72.39 128.27 0)
@@
 				)
 				(hide yes)
-			)
-		)
-		(property "PageName" ""
-			(at 179.705 556.26 0)
-			(effects
-				(font
-					(size 1.524 1.524)
-				)
-				(hide yes)

Commit message: populate stdc14
Parts:
- J6: now fitted
Changed lines of the file:
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@@
 		(in_bom yes)
 		(on_board yes)
-		(dnp yes)
+		(dnp no)
 		(property "Reference" "J6"
 			(at 281.94 52.0699 0)

Commit message: fix stdc - reroute power on pcb
Parts:
- D13, D9: LCSC (none) -> C2290
- J6: footprint dnt:SAMTEC_FTSH-107-01-F-DV-K-Fix -> dnt:Conn_SAMTEC_FTSH-107-01-F-DV-K-Fix
Changed lines of the file:
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@@
 			)
 		)
-		(property "Datasheet" "~"
+		(property "Datasheet" "https://jlcpcb.com/api/file/downloadByFileSystemAccessId/8550724001388785664"
 			(at 148.59 254 0)
 			(effects
@@
 		(property "Sim.Pins" "1=K 2=A"
 			(at 148.59 258.064 0)
+			(effects
+				(font
+					(size 1.27 1.27)
+				)
+				(hide yes)
+			)
+		)
+		(property "LCSC" "C2290"
+			(at 148.59 254 0)
 			(effects
 				(font
@@
 			)
 		)
-		(property "Footprint" "dnt:SAMTEC_FTSH-107-01-F-DV-K-Fix"
+		(property "Footprint" "dnt:Conn_SAMTEC_FTSH-107-01-F-DV-K-Fix"
 			(at 294.132 82.042 0)
 			(effects
@@
 	)
 	(symbol
-		(lib_name "LED-WHITE_1")
 		(lib_id "dnt_global:LED-WHITE")
 		(at 93.98 254 180)
@@
 			)
 		)
-		(property "Datasheet" "~"
+		(property "Datasheet" "https://jlcpcb.com/api/file/downloadByFileSystemAccessId/8550724001388785664"
 			(at 93.98 254 0)
 			(effects
@@
 			(effects
 				(font
+					(size 1.27 1.27)
+				)
+				(hide yes)
+			)
+		)
+		(property "LCSC" "C2290"
+			(at 93.98 254 0)
+			(effects
+				(font

Commit message: lcsc components and cleanup
Changed lines of the file:
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@@
 	(wire
 		(pts
-			(xy 107.95 88.9) (xy 111.76 88.9)
+			(xy 106.68 88.9) (xy 111.76 88.9)
 		)
 		(stroke
@@
 	(wire
 		(pts
-			(xy 107.95 80.01) (xy 107.95 88.9)
+			(xy 106.68 80.01) (xy 106.68 88.9)
 		)
 		(stroke
@@
 		)
 		(stroke
-			(width 0)
-			(type default)
-		)
-	)
-	(wire
-		(pts
-			(xy 106.68 80.01) (xy 107.95 80.01)
-		)
-		(stroke

Commit message: fix 10uf 25v
Parts:
- C22: footprint Capacitor_SMD:C_0603_1608Metric -> dnt:C_0603_1608Metric; symbol Device:C -> dnt_global:0603,10uF,_25V; Attrition Qty (none) -> 8; Capacitance (none) -> 10uF; Category (none) -> Capacitors,Multilayer Ceramic Capacitors MLCC - SMD/SMT; Class (none) -> Basic Component; Manufacturer (none) -> Samsung Electro-Mechanics; Minimum Qty (none) -> 20; Part (none) -> CL10A106MA8NRNC; Price (none) -> 0.021USD; Process (none) -> SMT; Stock (none) -> 3388297; Temperature Coefficient (none) -> X5R; Tolerance (none) -> ±20%; Voltage 25V -> (none); Voltage Rated (none) -> 25V
Changed lines of the file:
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@@
 	)
 	(symbol
-		(lib_id "Device:C")
+		(lib_id "dnt_global:0603,10uF,_25V")
 		(at 148.59 76.2 180)
 		(unit 1)
@@
 			)
 		)
-		(property "Footprint" "Capacitor_SMD:C_0603_1608Metric"
-			(at 147.6248 72.39 0)
+		(property "Footprint" "dnt:C_0603_1608Metric"
+			(at 150.368 76.2 90)
 			(effects
 				(font
@@
 			)
 		)
-		(property "Datasheet" "~"
+		(property "Datasheet" "https://www.lcsc.com/datasheet/lcsc_datasheet_2304140030_Samsung-Electro-Mechanics-CL10A106MA8NRNC_C96446.pdf"
 			(at 148.59 76.2 0)
 			(effects
@@
 			)
 		)
-		(property "Description" "Unpolarized capacitor"
-			(at 148.59 76.2 0)
-			(effects
-				(font
-					(size 1.27 1.27)
-				)
-				(hide yes)
-			)
-		)
-		(property "PN" ""
+		(property "Description" "25V 10uF X5R ±20% 0603 Multilayer Ceramic Capacitors MLCC - SMD/SMT ROHS"
 			(at 148.59 76.2 0)
 			(effects
@@
 			)
 		)
-		(property "Voltage" "25V"
-			(at 145.542 71.374 0)
-			(effects
-				(font
-					(size 1.27 1.27)
-				)
-			)
-		)
-		(property "Sim.Device" ""
+		(property "Stock" "3388297"
 			(at 148.59 76.2 0)
 			(effects
@@
 			)
 		)
-		(property "Sim.Pins" ""
+		(property "Price" "0.021USD"
 			(at 148.59 76.2 0)
 			(effects
@@
 			)
 		)
-		(property "Silkscreen" ""
+		(property "Process" "SMT"
 			(at 148.59 76.2 0)
 			(effects
+				(font
+					(size 1.27 1.27)
+				)
+				(hide yes)
+			)
+		)
+		(property "Minimum Qty" "20"
+			(at 148.59 76.2 0)
+			(effects
+				(font
+					(size 1.27 1.27)
+				)
+				(hide yes)
+			)
+		)
+		(property "Attrition Qty" "8"
+			(at 148.59 76.2 0)
+			(effects
+				(font
+					(size 1.27 1.27)
+				)
+				(hide yes)
+			)
+		)
+		(property "Class" "Basic Component"
+			(at 148.59 76.2 0)
+			(effects
+				(font
+					(size 1.27 1.27)
+				)
+				(hide yes)
+			)
+		)
+		(property "Category" "Capacitors,Multilayer Ceramic Capacitors MLCC - SMD/SMT"
+			(at 148.59 76.2 0)
+			(effects
+				(font
+					(size 1.27 1.27)
+				)
+				(hide yes)
+			)
+		)
+		(property "Manufacturer" "Samsung Electro-Mechanics"
+			(at 148.59 76.2 0)
+			(effects
+				(font
+					(size 1.27 1.27)
+				)
+				(hide yes)
+			)
+		)
+		(property "Part" "CL10A106MA8NRNC"
+			(at 148.59 76.2 0)
+			(effects
+				(font
+					(size 1.27 1.27)
+				)
+				(hide yes)
+			)
+		)
+		(property "Voltage Rated" "25V"
+			(at 146.558 74.1538 0)
+			(effects
+				(font
+					(size 0.8 0.8)
+				)
+				(justify left)
+			)
+		)
+		(property "Tolerance" "±20%"
+			(at 148.59 76.2 0)
+			(effects
+				(font
+					(size 1.27 1.27)
+				)
+				(hide yes)
+			)
+		)
+		(property "Capacitance" "10uF"
+			(at 148.59 76.2 0)
+			(effects
+				(font
+					(size 1.27 1.27)
+				)
+				(hide yes)
+			)
+		)
+		(property "Temperature Coefficient" "X5R"
+			(at 148.59 76.2 0)
+			(effects

Commit message: continue lssc fixups
Parts:
- C12, C13, C14, C15, C19, C20, C21, C24: footprint Capacitor_SMD:C_0603_1608Metric -> dnt:C_0603_1608Metric; symbol Device:C -> dnt_global:0603,100nF; Attrition Qty (none) -> 10; Capacitance (none) -> 100nF; Category (none) -> Capacitors,Multilayer Ceramic Capacitors MLCC - SMD/SMT; Class (none) -> Basic Component; Manufacturer (none) -> YAGEO; Minimum Qty (none) -> 20; Part (none) -> CC0603KRX7R9BB104; Price (none) -> 0.006USD; Process (none) -> SMT; Stock (none) -> 70324515; Temperature Coefficient (none) -> X7R; Tolerance (none) -> ±10%; Voltage Rated (none) -> 50V
- C18: footprint Capacitor_SMD:C_0603_1608Metric -> dnt:C_0603_1608Metric; symbol Device:C -> dnt_global:0603,100nF; Attrition Qty (none) -> 10; Capacitance (none) -> 100nF; Category (none) -> Capacitors,Multilayer Ceramic Capacitors MLCC - SMD/SMT; Class (none) -> Basic Component; Manufacturer (none) -> YAGEO; Minimum Qty (none) -> 20; Part (none) -> CC0603KRX7R9BB104; Price (none) -> 0.006USD; Process (none) -> SMT; Stock (none) -> 70324515; Temperature Coefficient (none) -> X7R; Tolerance (none) -> ±10%; Voltage 16V -> (none); Voltage Rated (none) -> 50V
Other:
- moved on the sheet: C12, C13, C14, C15, C18, C19, C20, C21

Commit message: lcsc changes done - export for prod
Parts:
- R12, R13, R14: footprint PCM_JLCPCB:R_0402 -> dnt:R_0402_1005Metric; symbol dnt_global:Resistor_0402,10kΩ -> dnt_global:0402,10kΩ
- R15, R16: symbol dnt_global:Resistor_0402,10kΩ -> PCM_JLCPCB-Resistors:0402,100Ω; LCSC C25744 -> C25076; Part 0402WGF1002TCE -> 0402WGF1000TCE; Resistance 10kΩ -> 100Ω; Stock 24372091 -> 5907585; Temperature Coefficient ±100ppm/°C -> ±200ppm/°C
- R17, R18, R19: value 100Ω -> 100R
Changed lines of the file:
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@@
 	)
 	(symbol
-		(lib_id "dnt_global:Resistor_0402,10kΩ")
+		(lib_id "dnt_global:0402,10kΩ")
 		(at 44.45 107.95 90)
 		(mirror x)
@@
 			)
 		)
-		(property "Footprint" "PCM_JLCPCB:R_0402"
+		(property "Footprint" "dnt:R_0402_1005Metric"
 			(at 44.45 106.172 90)
 			(effects
@@
 	)
 	(symbol
-		(lib_id "dnt_global:Resistor_0402,10kΩ")
+		(lib_id "dnt_global:0402,10kΩ")
 		(at 43.18 146.05 0)
 		(mirror x)
@@
 			)
 		)
-		(property "Footprint" "PCM_JLCPCB:R_0402"
+		(property "Footprint" "dnt:R_0402_1005Metric"
 			(at 41.402 146.05 90)
 			(effects
@@
 	)
 	(symbol
-		(lib_id "dnt_global:Resistor_0402,10kΩ")
+		(lib_id "PCM_JLCPCB-Resistors:0402,100Ω")
 		(at 290.83 124.46 0)
 		(unit 1)
@@
 			)
 		)
-		(property "Datasheet" "https://www.lcsc.com/datasheet/lcsc_datasheet_2411221126_UNI-ROYAL-Uniroyal-Elec-0402WGF1002TCE_C25744.pdf"
+		(property "Datasheet" "https://www.lcsc.com/datasheet/lcsc_datasheet_2205311900_UNI-ROYAL-Uniroyal-Elec-0402WGF1000TCE_C25076.pdf"
 			(at 290.83 124.46 0)
 			(effects
@@
 			)
 		)
-		(property "Description" "62.5mW Thick Film Resistors 50V ±100ppm/°C ±1% 10kΩ 0402 Chip Resistor - Surface Mount ROHS"
+		(property "Description" "62.5mW Thick Film Resistors 50V ±1% ±200ppm/°C 100Ω 0402 Chip Resistor - Surface Mount ROHS"
 			(at 290.83 124.46 0)
 			(effects
@@
 			)
 		)
-		(property "LCSC" "C25744"
+		(property "LCSC" "C25076"
 			(at 290.83 124.46 0)
 			(effects
@@
 			)
 		)
-		(property "Stock" "24372091"
+		(property "Stock" "5907585"
 			(at 290.83 124.46 0)
 			(effects
@@
 			)
 		)
-		(property "Part" "0402WGF1002TCE"
+		(property "Part" "0402WGF1000TCE"
 			(at 290.83 124.46 0)
 			(effects
@@
 			)
 		)
-		(property "Resistance" "10kΩ"
+		(property "Resistance" "100Ω"
 			(at 290.83 124.46 0)
 			(effects
@@
 			)
 		)
-		(property "Temperature Coefficient" "±100ppm/°C"
+		(property "Temperature Coefficient" "±200ppm/°C"
 			(at 290.83 124.46 0)
 			(effects
@@
 			)
 		)
-		(property "Value" "100Ω"
+		(property "Value" "100R"
 			(at 366.268 78.74 90)
 			(do_not_autoplace yes)
@@
 	)
 	(symbol
-		(lib_id "dnt_global:Resistor_0402,10kΩ")
+		(lib_id "PCM_JLCPCB-Resistors:0402,100Ω")
 		(at 290.83 74.93 0)
 		(unit 1)
@@
 			)
 		)
-		(property "Datasheet" "https://www.lcsc.com/datasheet/lcsc_datasheet_2411221126_UNI-ROYAL-Uniroyal-Elec-0402WGF1002TCE_C25744.pdf"
+		(property "Datasheet" "https://www.lcsc.com/datasheet/lcsc_datasheet_2205311900_UNI-ROYAL-Uniroyal-Elec-0402WGF1000TCE_C25076.pdf"
 			(at 290.83 74.93 0)
 			(effects
@@
 			)
 		)
-		(property "Description" "62.5mW Thick Film Resistors 50V ±100ppm/°C ±1% 10kΩ 0402 Chip Resistor - Surface Mount ROHS"
+		(property "Description" "62.5mW Thick Film Resistors 50V ±1% ±200ppm/°C 100Ω 0402 Chip Resistor - Surface Mount ROHS"
 			(at 290.83 74.93 0)
 			(effects
@@
 			)
 		)
-		(property "LCSC" "C25744"
+		(property "LCSC" "C25076"
 			(at 290.83 74.93 0)
 			(effects
@@
 			)
 		)
-		(property "Stock" "24372091"
+		(property "Stock" "5907585"
 			(at 290.83 74.93 0)
 			(effects
@@
 			)
 		)
-		(property "Part" "0402WGF1002TCE"
+		(property "Part" "0402WGF1000TCE"
 			(at 290.83 74.93 0)
 			(effects
@@
 			)
 		)
-		(property "Resistance" "10kΩ"
+		(property "Resistance" "100Ω"
 			(at 290.83 74.93 0)
 			(effects
@@
 			)
 		)
-		(property "Temperature Coefficient" "±100ppm/°C"
+		(property "Temperature Coefficient" "±200ppm/°C"
 			(at 290.83 74.93 0)
 			(effects
@@
 			)
 		)
-		(property "Value" "100Ω"
+		(property "Value" "100R"
 			(at 332.74 76.454 90)
 			(do_not_autoplace yes)
@@
 			)
 		)
-		(property "Value" "100Ω"
+		(property "Value" "100R"
 			(at 322.58 76.2 90)
 			(do_not_autoplace yes)
@@
 	)
 	(symbol
-		(lib_id "dnt_global:Resistor_0402,10kΩ")
+		(lib_id "dnt_global:0402,10kΩ")
 		(at 250.19 160.02 0)
 		(mirror x)
@@
 			)
 		)
-		(property "Footprint" "PCM_JLCPCB:R_0402"
+		(property "Footprint" "dnt:R_0402_1005Metric"
 			(at 248.412 160.02 90)
 			(effects
