File: z9-console/stm32.kicad_sch (KiCad schematic)
At the start: 75 parts, among them J6 ST_STDC14 - SAMTEC_FTSH-107-0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, J7 TC2070 - TAG Connect, SW2 SW_Push, SW3 SW_Push, U8 STM32F427V_G-I_Tx, X2 8MHz 20pF

Commit message: more change - generarte jlc
Parts:
- C11: symbol dnt_global:0402,100nF, 16V -> PCM_JLCPCB-Capacitors:0402,10nF; Capacitance 100nF -> 10nF; LCSC C1525 -> C15195; Part CL05B104KO5NNNC -> CL05B103KB5NNNC; Price 0.004USD -> 0.005USD; Stock 20208285 -> 4779042; Voltage Rated 16V -> 50V
- D11, D12, D15, D8: footprint dnt:LED_0603_1608Metric - polarity -> PCM_JLCPCB:D_0603; symbol dnt_global:LED-YELLOW -> dnt_global:LED,0603,Yellow; Attrition Qty (none) -> 6; Category (none) -> Optoelectronics,Light Emitting Diodes (LED); Class (none) -> Preferred Component; Dominant Wavelength (none) -> 586nm~595nm; Emitted Color (none) -> Yellow; Forward Current (none) -> 25mA; Forward Voltage (VF) (none) -> 1.6V~2.6V; JLCPCB Rotation Offset 0 -> (none); LCSC C72038 -> C89811; Lens Color (none) -> Colorless Transparent Lens; Luminous Intensity (none) -> 100mcd~220mcd; Manufacturer (none) -> Foshan NationStar Optoelectronics; Minimum Qty (none) -> 20; Operating Temperature (none) -> -30°C~+85°C; Part (none) -> NCD0603Y2; Power Dissipation (none) -> 65mW; Price (none) -> 0.021USD; Process (none) -> SMT; Stock (none) -> 109176; Viewing Angle (none) -> 130°

Commit message: sheet updates
Other:
- company: DNT -> Zero9 -  0-9.au
- title: l8-console -> (none)
Changed lines of the file:
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@@
 	(paper "A3")
 	(title_block
-		(title "l8-console")
 		(date "2022-04-10")
-		(company "DNT")
+		(company "Zero9 -  0-9.au")
+		(comment 1 "Some schematic is shared ")
 	)
 	(text "SPI1 40MHZ\nSPI2 20MHz\nSPI3 20MHz \nSPI4 40MHz"
