File: z9-console/sensor.kicad_sch (KiCad schematic)
At the start: 17 parts, among them U10 ISM330DHCX, U11 ST_SENSOR_2

Commit message: lcsc changes done - export for prod
Parts:
- R21, R22, R23, R24, R25, R26, R27: footprint PCM_JLCPCB:R_0402 -> dnt:R_0402_1005Metric; symbol dnt_global:Resistor_0402,10kΩ -> dnt_global:0402,10kΩ
Changed lines of the file:
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@@
 	)
 	(symbol
-		(lib_id "dnt_global:Resistor_0402,10kΩ")
+		(lib_id "dnt_global:0402,10kΩ")
 		(at 88.9 114.3 0)
 		(mirror x)
@@
 			)
 		)
-		(property "Footprint" "PCM_JLCPCB:R_0402"
+		(property "Footprint" "dnt:R_0402_1005Metric"
 			(at 87.122 114.3 90)
 			(effects
@@
 	)
 	(symbol
-		(lib_id "dnt_global:Resistor_0402,10kΩ")
+		(lib_id "dnt_global:0402,10kΩ")
 		(at 83.82 114.3 0)
 		(mirror x)
@@
 			)
 		)
-		(property "Footprint" "PCM_JLCPCB:R_0402"
+		(property "Footprint" "dnt:R_0402_1005Metric"
 			(at 82.042 114.3 90)
 			(effects
@@
 	)
 	(symbol
-		(lib_id "dnt_global:Resistor_0402,10kΩ")
+		(lib_id "dnt_global:0402,10kΩ")
 		(at 64.77 41.91 0)
 		(mirror x)
@@
 			)
 		)
-		(property "Footprint" "PCM_JLCPCB:R_0402"
+		(property "Footprint" "dnt:R_0402_1005Metric"
 			(at 62.992 41.91 90)
 			(effects
@@
 	)
 	(symbol
-		(lib_id "dnt_global:Resistor_0402,10kΩ")
+		(lib_id "dnt_global:0402,10kΩ")
 		(at 250.19 87.63 0)
 		(mirror x)
@@
 			)
 		)
-		(property "Footprint" "PCM_JLCPCB:R_0402"
+		(property "Footprint" "dnt:R_0402_1005Metric"
 			(at 248.412 87.63 90)
 			(effects
@@
 	)
 	(symbol
-		(lib_id "dnt_global:Resistor_0402,10kΩ")
+		(lib_id "dnt_global:0402,10kΩ")
 		(at 245.11 87.63 0)
 		(mirror x)
@@
 			)
 		)
-		(property "Footprint" "PCM_JLCPCB:R_0402"
+		(property "Footprint" "dnt:R_0402_1005Metric"
 			(at 243.332 87.63 90)
 			(effects
@@
 	)
 	(symbol
-		(lib_id "dnt_global:Resistor_0402,10kΩ")
+		(lib_id "dnt_global:0402,10kΩ")
 		(at 283.21 62.23 0)
 		(mirror x)
@@
 			)
 		)
-		(property "Footprint" "PCM_JLCPCB:R_0402"
+		(property "Footprint" "dnt:R_0402_1005Metric"
 			(at 281.432 62.23 90)
 			(effects
@@
 	)
 	(symbol
-		(lib_id "dnt_global:Resistor_0402,10kΩ")
+		(lib_id "dnt_global:0402,10kΩ")
 		(at 260.35 59.69 0)
 		(mirror x)
@@
 			)
 		)
-		(property "Footprint" "PCM_JLCPCB:R_0402"
+		(property "Footprint" "dnt:R_0402_1005Metric"
 			(at 258.572 59.69 90)
 			(effects

Commit message: more change - generarte jlc
Parts:
- U10: JLCPCB Rotation Offset (none) -> 180
Changed lines of the file:
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@@
+			)
+		)
+		(property "JLCPCB Rotation Offset" "180"
+			(at 118.11 66.04 0)
+			(effects
+				(font
+					(size 1.27 1.27)
+				)
+				(hide yes)
 			)
 		)
