File: z9-console/sensor.kicad_sch (KiCad schematic)
At the start: 17 parts, among them U10 ISM330DHCX, U11 ST_SENSOR_2

Commit message: more moving offset to library - tedious
Parts:
- U10: FT Rototation Offset (none) -> 180; JLCPCB Rotation Offset 180 -> (none)
Changed lines of the file:
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@@
 		)
 		(property "Description" "iNEMO inertial module with embedded Machine Learning Core: always-on 3D accelerometer and 3D gyroscope with digital output for industrial applications, LGA-14"
-			(at 119.38 60.96 0)
+			(at 118.618 37.084 0)
 			(effects
 				(font
@@
 			)
 		)
-		(property "JLCPCB Rotation Offset" "180"
+		(property "FT Rototation Offset" "180"
 			(at 118.11 66.04 0)
 			(effects

Commit message: ism issues
Parts:
- U: renamed from U10; FT Rotation Offset (none) -> 180; FT Rototation Offset 180 -> (none)
Changed lines of the file:
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@@
 		(dnp no)
 		(fields_autoplaced yes)
-		(property "Reference" "U10"
+		(property "Reference" "U"
 			(at 120.2533 83.82 0)
 			(effects
@@
 			)
 		)
-		(property "FT Rototation Offset" "180"
+		(property "FT Rotation Offset" "180"
 			(at 118.11 66.04 0)
 			(effects
@@
 			(project ""
 				(path "/8d063f79-9282-4820-bcf4-1ff3c006cf08/801ffdec-7184-42a0-bbdb-64e97598ca97"
-					(reference "U10")
+					(reference "U")
 					(unit 1)
 				)

Commit message: submitted to jlcpcb 00:23 1/10/20025
Parts:
- renumbered U to U9
Changed lines of the file:
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@@
 		(dnp no)
 		(fields_autoplaced yes)
-		(property "Reference" "U"
+		(property "Reference" "U9"
 			(at 120.2533 83.82 0)
 			(effects
@@
 			(project ""
 				(path "/8d063f79-9282-4820-bcf4-1ff3c006cf08/801ffdec-7184-42a0-bbdb-64e97598ca97"
-					(reference "U")
+					(reference "U9")
 					(unit 1)
 				)

Commit message: sheet updates
Other:
- company: (none) -> Zero9 -  0-9.au
Changed lines of the file:
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@@
 	(generator "eeschema")
 	(generator_version "9.0")
-	(paper "A3")
+	(paper "A4")
+	(title_block
+		(company "Zero9 -  0-9.au")
+		(comment 1 "Some schematic is shared ")
+	)
 	(junction
 		(at 132.08 58.42)
