File: z9-console/z9-console.kicad_pcb (KiCad board)
At the start: 2 copper layers, 89.5 x 55.5 mm, 130 parts, among them J10 Screw_Terminal_01x06, J2 LCD 3.2" 240x320 Conn_01x14_P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, J4 Conn_01x04_Pin, J6 ST_STDC14 - SAMTEC_FTSH-107-0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, J7 TC2070 - TAG Connect, J801 USB_C_Receptacle_USB2.0_16P, J9 JST GH, Q701 AO3400A, SW2 SW_Push, SW3 SW_Push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

Commit message: continue lssc fixups
Parts:
- C12, C13, C14, C15, C18, C19, C2, C20, C21, C22, C24, C29, C3, C7, C8, C9: footprint Capacitor_SMD:C_0603_1608Metric -> dnt:C_0603_1608Metric
- C701, C951, C952, C953: footprint PCM_JLCPCB:C_0603 -> dnt:C_0603_1608Metric
- R10, R12, R13, R14, R2, R20, R21, R22, R23, R24, R25, R26, R27, R3, R4, R5, R804: footprint PCM_JLCPCB:R_0402 -> dnt:R_0402_1005Metric
- R702: footprint PCM_JLCPCB:R_0603 -> dnt:R_0402_1005Metric
- moved R9 0.96 mm to (106.1, 75.2)
- moved C9 0.91 mm to (105.9, 77.4), turned to -90 degrees
- moved R10 0.66 mm to (106.1, 74.1)
- moved R702 0.28 mm to (119.7, 123.4)
Routing:
- net Net-(D6-K): track 3.29 -> 0.00 mm
- net Net-(U7-CB): track 4.25 -> 2.26 mm
- net Net-(C10-Pad1): track 13.6 -> 15.2 mm
- net GND: track 21.7 -> 20.9 mm
- net Net-(U7-FB): track 3.68 -> 2.96 mm

Commit message: more change - generarte jlc
Parts:
- D11, D12, D15, D8: footprint dnt:LED_0603_1608Metric - polarity -> PCM_JLCPCB:D_0603
- Q701: footprint Package_TO_SOT_SMD:SOT-23 -> PCM_JLCPCB:Q_SOT-23
- R17, R18, R19: value 100Ω -> 100R
- R701: value 100Ω -> 100R; footprint PCM_JLCPCB:R_0603 -> PCM_JLCPCB:R_0402
- R702: value 10kΩ -> 10K
- R805: value 2.2kΩ -> 2.2k
- moved R701 2.48 mm to (118.2, 123.1)
- moved R702 0.87 mm to (120.5, 123.1)
- moved Q701 0.28 mm to (119.3, 120.7)
Routing:
- net Net-(Q701-G): track 6.97 -> 6.19 mm

Commit message: ism issues
Parts:
- D6: value MicroSMP(DO-219AD) -> V1P6-M3/H 60V 1A
- R9: value 54K9 -> 56K
Changed lines of the file:
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@@
 			)
 		)
-		(property "FT Rototation Offset" "180"
+		(property "FT Rotatation Offset" "180"
 			(at 0 0 180)
 			(unlocked yes)
@@
 			)
 		)
-		(property "Value" "54K9"
+		(property "Value" "56K"
 			(at 0 0.2 180)
 			(layer "F.Fab")
@@
 			)
 		)
+		(property "FT Rotation Offset" "180"
+			(at 0 0 0)
+			(unlocked yes)
+			(layer "F.Fab")
+			(hide yes)
+			(effects
+				(font
+					(size 1 1)
+					(thickness 0.15)
+				)
+			)
+		)
 		(property ki_fp_filters "Q_*")
 		(sheetname "/shared buzzer/")
@@
 			)
 		)
-		(property "Value" "MicroSMP(DO-219AD)"
+		(property "Value" "V1P6-M3/H 60V 1A"
 			(at 0 1.65 180)
 			(unlocked yes)

Commit message: submitted to jlcpcb 00:23 1/10/20025
Parts:
- renumbered U10 to U9
Changed lines of the file:
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@@
 	(net 136 "unconnected-(U5-EN-Pad4)")
 	(net 137 "unconnected-(U6-NC-Pad8)")
-	(net 138 "unconnected-(U10-OCS_AUX-Pad10)")
+	(net 138 "unconnected-(U9-OCS_AUX-Pad10)")
 	(net 139 "unconnected-(U11-Pad9)")
 	(net 140 "unconnected-(U11-Pad7)")
@@
 		(descr "LGA, 14 Pin (https://www.st.com/resource/en/datasheet/lsm6ds3tr-c.pdf), generated with kicad-footprint-generator ipc_noLead_generator.py")
 		(tags "LGA NoLead")
-		(property "Reference" "U10"
+		(property "Reference" "U9"
 			(at 4.5 -1.9375 0)
 			(layer "F.SilkS")
@@
 			)
 		)
+		(property "FT Rotation Offset" "180"
+			(at 0 0 180)
+			(unlocked yes)
+			(layer "F.Fab")
+			(hide yes)
+			(effects
+				(font
+					(size 1 1)
+					(thickness 0.15)
+				)
+			)
+		)
 		(property ki_fp_filters "*LGA*3x2.5mm*P0.5mm*LayoutBorder3x4y*")
 		(sheetname "/sensor/")
@@
 			(layers "F.Cu" "F.Mask" "F.Paste")
 			(roundrect_rratio 0.25)
-			(net 138 "unconnected-(U10-OCS_AUX-Pad10)")
+			(net 138 "unconnected-(U9-OCS_AUX-Pad10)")
 			(pinfunction "OCS_AUX")
 			(pintype "passive+no_connect")
