File: z9-console/power.kicad_sch (KiCad schematic)
At the start: 29 parts, among them U5 TLV76733DRVx, U6 B0505XT-1WR3, U7 LMR14006YDDCR

Commit message: add image - start shared ps
Parts:
- removed C10, C5: 22uF, Capacitor_SMD:C_0805_2012Metric, symbol Device:C
- removed C2, C3, C7: 10uF, dnt:C_0603_1608Metric, symbol dnt_global:0603,10uF,_25V
- removed C4: 1uF, Capacitor_SMD:C_0603_1608Metric, symbol Device:C
- removed C6: 10uF, Capacitor_SMD:C_0805_2012Metric, symbol Device:C
- removed C8, C9: 100nF, dnt:C_0603_1608Metric, symbol dnt_global:0603,100nF
- removed D2: SS54, dnt:D_SMA - polarity, symbol dnt_global:Diode_SS54
- removed D3: SM15T100CA, Diode_SMD:D_SMC, symbol Device:D_TVS
- removed D4, D5, D7: LED-RED, dnt:LED_0603_1608Metric - polarity, symbol dnt_global:LED-RED
- removed D6: V1P6-M3/H 60V 1A, Diode_SMD:D_MicroSMP_AK, symbol dnt_global:Diode - V1P6-M3/H 60V 1A Schotty
- removed F2, F3, F4: Fuse, Fuse:Fuse_0805_2012Metric, symbol dnt_global:Fuse_16V_500mA_100A_1A_150mΩ_0805_PTC_Resettable_Fuses_ROHS
- removed L2: 3.3uH, Inductor_SMD:L_Sunlord_SWPA4030S, symbol Device:L_Ferrite
- removed R10: 10K, dnt:R_0402_1005Metric, symbol dnt_global:0402,10kΩ
- removed R11, R7, R8: 2.2K, PCM_JLCPCB:R_0402, symbol PCM_JLCPCB-Resistors:0402,2.2kΩ
- removed R9: 56K, PCM_JLCPCB:R_0402, symbol PCM_JLCPCB-Resistors:0402,56kΩ
- removed TP2: +3.3V, dnt:TestPoint_Pad_D1.0mm FP .6R, symbol Connector:TestPoint
- removed TP3: 5V, dnt:TestPoint_Pad_D1.0mm FP .6R, symbol Connector:TestPoint
- removed U5: TLV76733DRVx, Package_SON:WSON-6-1EP_2x2mm_P0.65mm_EP1x1.6mm_ThermalVias, symbol dnt_global:TLV76733DRVx
- removed U6: B0505XT-1WR3, dnt:B0505_Isolated_SMD, symbol dnt_global:B0505_Isolated_SMD
- removed U7: LMR14006YDDCR, Package_TO_SOT_SMD:SOT-23-6, symbol dnt_global:LMR14006YDDCR
Connections:
- no-connect marks 1 -> 0
Other:
- note removed: "Load Dump TVS"
- note removed: "todo - reverse feed in here from USB - needs protection"
