File: z9-console/power.kicad_sch (KiCad schematic)
At the start: 0 parts

Commit message: sheet updates
Other:
- company: (none) -> Zero9 -  0-9.au
Changed lines of the file:
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@@
 	(generator_version "9.0")
 	(paper "A4")
+	(title_block
+		(company "Zero9 -  0-9.au")
+		(comment 1 "Some schematic is shared ")
+	)
 )
