File: z9-console/untitled.kicad_sch (KiCad schematic)
At the start: 29 parts, among them U301 TLV76733DRVx, U302 B0505XT-1WR3, U303 LMR14006YDDCR

Commit message: sheet updates
Other:
- company: (none) -> Zero9 -  0-9.au
Changed lines of the file:
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@@
 	(generator_version "9.0")
 	(paper "A4")
+	(title_block
+		(rev "v0.0.3")
+		(company "Zero9 -  0-9.au")
+		(comment 1 "Some schematic is shared ")
+	)
 	(text "Load Dump TVS\n\n"
 		(exclude_from_sim no)
