File: z9-console/z9-console.kicad_sch (KiCad schematic)
At the start: 4 parts

Commit message: add image - start shared ps
Other:
- added sheet shared ps (untitled.kicad_sch)
Changed lines of the file:
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@@
+	)
+	(sheet
+		(at 162.56 30.48)
+		(size 88.9 45.72)
+		(exclude_from_sim no)
+		(in_bom yes)
+		(on_board yes)
+		(dnp no)
+		(fields_autoplaced yes)
+		(stroke
+			(width 0.1524)
+			(type solid)
+		)
+		(fill
+			(color 0 0 0 0.0000)
+		)
+		(property "Sheetname" "shared ps"
+			(at 162.56 29.7684 0)
+			(effects
+				(font
+					(size 1.27 1.27)
+				)
+				(justify left bottom)
+			)
+		)
+		(property "Sheetfile" "untitled.kicad_sch"
+			(at 162.56 76.7846 0)
+			(effects
+				(font
+					(size 1.27 1.27)
+				)
+				(justify left top)
+			)
+		)
+		(instances
+			(project "z9-console"
+				(path "/8d063f79-9282-4820-bcf4-1ff3c006cf08"
+					(page "10")
+				)
+			)
+		)
 	)
 	(sheet

Commit message: sheet updates
Other:
- company: (none) -> Zero9 -  0-9.au
Changed lines of the file:
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@@
 	(title_block
 		(date "2024-05-30")
+		(company "Zero9 -  0-9.au")
+		(comment 1 "Some schematic is shared ")
 	)
 	(rectangle
